File: pc2_key.brd (EAGLE design)
At the start: 100 x 26 mm, 25 parts, among them IC1 4011D, IC2 MC34063AD

Commit message: 2
Parts:
- removed 1C10: 220u/6V, resistor:E3,5-8
- removed 1R15: 27K, resistor:R0805
- removed 2D1: 1N5819, diode:DO41-10
- removed 2L1: 220uH, inductor-neosid:SD12_1000
- removed 2R2: 180R, resistor:R0805
- removed C14: 100n, resistor:C0805K
- removed C16: 50u, resistor:E2,5-6
- removed IC1: 4011D, 40xx:SO14
- removed IC2: MC34063AD, mc34063:SOIC8
- added C1: 10m, rcl:C1210
- added C3, C4: 100n, resistor:C0805K
- added D1: (no value), diode:SMB
- added D10, D11, D12, D13, D14, D15, D6, D8, D9: (no value), diode:SOD80C
- added DA1: MC34063AD, mc34063:SOIC8
- added DD1: 4011D, 40xx:SO14
- added L1: 100u, rcl:6000-XXXX-RC
- added R10, R11, R12, R7, R8, R9: (no value), rcl:R0805
- 2C2: value 0.47n -> 59
- 2R1: value 1R -> 2r5
- 2R3: value 18K -> 11k
- 2R4: value 56K -> 18k
- C2: value 100n -> 10m; device resistor:C0805K -> rcl:C1210
- moved R3 119.4 mm to (2.54, -15.2), turned to 270 degrees
- moved R4 118.4 mm to (17.8, -40.6), turned to 90 degrees
- moved R2 113.2 mm to (-1.27, -15.2), turned to 270 degrees
- moved R1 106.9 mm to (-5.08, -15.2), turned to 270 degrees
- moved R5 105.1 mm to (-7.62, -35.6), turned to 90 degrees
- moved 2R3 103.6 mm to (-24.1, 40.6)
- moved 2R4 103.6 mm to (-19.1, 40.6)
- moved C15 103.6 mm to (-24.1, 35.6)
- moved R6 103.3 mm to (-7.62, -43.2), turned to 90 degrees
- moved VT3 100.8 mm to (7.62, -27.9)
- moved 2R1 97.0 mm to (0.00, 38.1), turned to 90 degrees
- moved 2C2 96.8 mm to (-11.4, 30.5), turned to 270 degrees
- moved C2 88.2 mm to (-48.3, 40.6), turned to 90 degrees
- moved VT2 85.9 mm to (-3.81, -30.5), turned to 180 degrees
- moved VT1 73.3 mm to (-14.0, -30.5), turned to 270 degrees
Connections:
- removed net +5V: 1C10.+, 1R15.1, 2D1.C, 2R4.2, C14.1
- removed net N$11: 1R15.2, C2.1
- removed net N$21: 2D1.A, 2L1.2, IC2.1
- removed net N$22: 2R2.2, IC2.8
- removed net N$24: 2L1.1, 2R1.2, 2R2.1, IC2.7
- removed net V+: 2R1.1, C15.1, C16.+, IC2.6
- removed net VDD: IC1.14
- removed net VSS: IC1.7
- new net +12V: 2R1.1, C15.1, C2.1, DA1.6
- new net N$13: R11.1, R2.1, R8.1, S1.D2
- new net N$14: R12.1, R3.1, R9.1, S1.D4
- new net N$15: D12.C, R9.2
- new net N$16: D11.C, R8.2
- new net N$17: D10.C, R7.2
- new net N$18: D15.C, R12.2
- new net N$20: D14.C, R11.2
- new net N$23: D13.C, R10.2
- new net N$26: D13.A, D14.A, D15.A, VT1.2
- new net N$27: D10.A, D11.A, D12.A, VT2.2
- new net N$28: D6.A, D8.A, D9.A, VT3.2
- net +3V3: now also 2R4.2, C1.1, C3.1, C4.1, DD1.14, L1.2
- net GND: now also C1.2, C2.2, C3.2, C4.2, D1.A, DA1.4, DD1.7; no longer C16.-, IC2.2, IC2.4
- net N$19: now also D1.C, DA1.2, L1.1; no longer 2C2.1, IC2.3
- net N$25: now also DA1.5; no longer IC2.5
- net N$3: now also 2R1.2, DA1.1, DA1.7, DA1.8; no longer R1.2, VT1.2
- net N$4: now also R1.1, R10.1, R7.1, S1.D1; no longer R2.2, VT2.2
- net N$5: now also 2C2.1, DA1.3; no longer R3.2, VT3.2
- net N$6: now also D9.C, R3.2; no longer R1.1, S1.D1
- net N$7: now also D8.C, R2.2; no longer R2.1, S1.D2
- net N$8: now also D6.C, R1.2; no longer R3.1, S1.D4
Routing:
- net N$4: track 0.00 -> 36.8 mm, vias 0 -> 1
- net N$13: track 0.00 -> 30.5 mm, vias 0 -> 1
- net N$14: track 0.00 -> 24.1 mm
- net GND: track 0.00 -> 14.0 mm
- net N$26: track 0.00 -> 7.62 mm
- net N$3: track 0.00 -> 6.47 mm
- net N$23: track 0.00 -> 2.43 mm
- net N$20: track 0.00 -> 2.43 mm
- net N$18: track 0.00 -> 2.43 mm

Commit message: 3
Parts:
- added 2C1: 59, resistor:C0805K
- added JP1, JP2: (no value), pinhead:1X02
- moved DD1 86.0 mm to (26.7, -3.81)
- moved C4 78.9 mm to (27.3, 5.08)
- moved L1 68.2 mm to (21.0, 11.4)
- moved D1 50.2 mm to (18.4, 8.26), turned to 90 degrees
- moved 2R3 49.5 mm to (17.1, 13.3), turned to 90 degrees
- moved 2R4 44.6 mm to (18.4, 16.5)
- moved C2 39.1 mm to (-27.3, 7.62), turned to 180 degrees
- moved 2C2 34.2 mm to (14.0, 7.62), turned to 0 degrees
- moved C15 31.9 mm to (-27.3, 3.81), turned to 180 degrees
- moved DA1 25.6 mm to (12.7, 13.3), turned to 0 degrees
- moved 2R1 25.5 mm to (8.26, 14.0), turned to 270 degrees
- moved C1 24.4 mm to (-33.0, 49.5)
- moved C3 18.3 mm to (-29.2, 49.5)
Connections:
- new net N$21: JP2.1, S1.SW2
- new net N$22: JP2.2, S1.SW1
- net +12V: now also JP1.1
- net GND: now also 2C1.2, JP1.2
- net N$5: now also 2C1.1
Routing:
- net GND: track 14.0 -> 83.1 mm
- net +12V: track 0.00 -> 57.9 mm
- net N$19: track 0.00 -> 21.2 mm
- net +3V3: track 0.00 -> 13.3 mm
- net N$22: track 0.00 -> 7.25 mm
- net N$21: track 0.00 -> 5.76 mm
- net N$25: track 0.00 -> 5.45 mm
- net N$3: track 6.47 -> 9.95 mm
Other:
- board size 100 x 26 mm -> 100 x 33 mm

Commit message: 4
Parts:
- moved R4 80.5 mm to (-22.2, 29.2)
- moved R6 76.9 mm to (-36.8, 27.9)
- moved C3 72.1 mm to (28.6, 6.35), turned to 180 degrees
- moved R5 72.1 mm to (-45.1, 26.0)
- moved VT2 72.1 mm to (-41.3, 31.1), turned to 270 degrees
- moved C1 71.5 mm to (26.7, 10.2), turned to 270 degrees
- moved VT3 66.6 mm to (-17.8, 33.7), turned to 270 degrees
- moved VT1 66.5 mm to (-33.7, 33.0)
- moved D6 38.3 mm to (-22.2, 14.0), turned to 180 degrees
- moved D9 38.3 mm to (-22.2, 8.89), turned to 180 degrees
- moved D8 38.0 mm to (-22.2, 11.4), turned to 180 degrees
- moved R1 31.6 mm to (-17.1, 14.0), turned to 180 degrees
- moved R3 31.1 mm to (-17.1, 8.89), turned to 180 degrees
- moved R2 31.0 mm to (-17.1, 11.4), turned to 180 degrees
- moved D13 27.3 mm to (-22.2, 5.71), turned to 180 degrees
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Connections:
- removed net N$17: D10.C, R7.2
- new net N$11: D10.A, R7.1
- net N$13: now also D11.C; no longer R8.1
- net N$16: now also D11.A, R8.1; no longer D11.C, R8.2
- net N$27: now also R7.2, R8.2; no longer D10.A, D11.A
- net N$4: now also D10.C; no longer R7.1
Routing:
- net +12V: track 57.9 -> 10.4 mm
- net N$14: track 24.1 -> 45.5 mm, vias 0 -> 2
- net GND: track 83.1 -> 66.7 mm
- net N$13: track 30.5 -> 38.7 mm, vias 1 -> 2
- net N$5: track 0.00 -> 6.44 mm
- net N$28: track 0.00 -> 5.08 mm
- net +3V3: track 13.3 -> 17.8 mm
- net N$26: track 7.62 -> 5.08 mm
- net N$8: track 0.00 -> 2.43 mm
- net N$7: track 0.00 -> 2.43 mm
- net N$6: track 0.00 -> 2.43 mm
- net N$15: track 0.00 -> 2.43 mm
- net N$25: track 5.45 -> 6.79 mm
- net N$4: track 36.8 -> 38.0 mm
- net N$3: track 9.95 -> 9.01 mm
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
Commit message: 6
Parts:
- moved D8 10.6 mm to (-13.3, 5.71), turned to 90 degrees
- moved R1 5.71 mm to (-22.9, 14.0)
- moved R10 5.71 mm to (-22.9, 5.71)
- moved R11 5.71 mm to (-22.9, 3.17)
- moved R12 5.71 mm to (-22.9, 0.64)
- moved R2 5.71 mm to (-22.9, 11.4)
- moved R3 5.71 mm to (-22.9, 8.89)
- moved R9 5.71 mm to (-22.9, -7.62)
- moved D12 4.45 mm to (-17.8, -7.62)
- moved D13 4.45 mm to (-17.8, 5.71)
- moved D14 4.45 mm to (-17.8, 3.17)
- moved D15 4.45 mm to (-17.8, 0.64)
- moved D6 4.45 mm to (-17.8, 14.0)
- moved D9 4.45 mm to (-17.8, 8.89)
- moved C2 2.54 mm to (-5.71, 14.0)
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Connections:
- removed net N$23: D13.C, R10.2
- new net N$17: D15.A, R12.1
- net N$13: now also D14.C, D8.C; no longer R11.1, R2.1
- net N$14: now also D12.C, D15.C, D9.C; no longer R12.1, R3.1, R9.1
- net N$15: now also D12.A, R9.1; no longer D12.C, R9.2
- net N$18: now also D14.A, R11.1; no longer D15.C, R12.2
- net N$20: now also D13.A, R10.1; no longer D14.C, R11.2
- net N$26: now also R10.2, R11.2, R12.2; no longer D13.A, D14.A, D15.A
- net N$27: now also R9.2; no longer D12.A
- net N$28: now also R1.2, R2.2, R3.2; no longer D6.A, D8.A, D9.A
- net N$4: now also D13.C, D6.C; no longer R1.1, R10.1
- net N$6: now also D9.A, R3.1; no longer D9.C, R3.2
- net N$7: now also D8.A, R2.1; no longer D8.C, R2.2
- net N$8: now also D6.A, R1.1; no longer D6.C, R1.2
Routing:
- net N$13: track 38.7 -> 28.3 mm, vias 2 -> 0
- net N$7: track 2.43 -> 12.6 mm
- net N$16: track 0.00 -> 6.24 mm
- net N$27: track 0.00 -> 5.08 mm
- net N$4: track 38.0 -> 40.7 mm
- net N$23: track 2.43 -> 0.00 mm
- net N$17: track 0.00 -> 2.43 mm
- net N$11: track 0.00 -> 2.43 mm
- net GND: track 66.7 -> 65.8 mm
- net N$14: track 45.5 -> 45.3 mm, vias 2 -> 0

Commit message: 7
Parts:
- added 2R2: 2r5, resistor:R0805
- added R13: 10, rcl:R0805
- added R14: (no value), rcl:R1206W
- R4, R6: device rcl:R0805 -> rcl:R1206W
- VT1, VT2, VT3: device m_transistor:TO126V -> m_transistor:TO92
- moved R5 80.5 mm to (34.6, 14.9), turned to 180 degrees
- moved VT2 69.4 mm to (26.4, 15.6), turned to 90 degrees
- moved R6 58.5 mm to (19.7, 13.0)
- moved VT1 52.5 mm to (15.9, 15.6), turned to 90 degrees
- moved R4 50.0 mm to (25.1, 13.0)
- moved VT3 42.8 mm to (21.0, 15.6), turned to 90 degrees
- moved DD1 26.1 mm to (43.8, 13.3), turned to 90 degrees
- moved C15 19.7 mm to (13.3, 11.1), turned to 90 degrees
- moved 2R4 17.6 mm to (24.4, 0.00)
- moved C4 16.9 mm to (43.5, 7.30), turned to 0 degrees
- moved L1 15.6 mm to (24.8, -5.08)
- moved C2 15.5 mm to (9.53, 11.4), turned to 90 degrees
- moved JP1 14.1 mm to (5.08, 13.3), turned to 0 degrees
- moved 2C1 12.2 mm to (17.1, -7.30)
- moved 2C2 12.2 mm to (17.1, -4.76)
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Connections:
- new net N$23: R13.2, S1.D3
- new net N$24: D10.C, R14.2
- new net OUT1: DD1.10, R4.1
- new net OUT2: DD1.11, DD1.8, R5.1
- new net OUT3: DD1.13, DD1.4, DD1.9, R6.1
- new net POWER: DD1.12
- new net SSD: DD1.5, DD1.6
- net +12V: now also 2R2.1
- net GND: now also R13.1; no longer S1.D3
- net N$10: now also VT2.2; no longer VT2.3
- net N$12: now also VT3.2; no longer VT3.3
- net N$26: now also VT1.3; no longer VT1.2
- net N$27: now also VT2.3; no longer VT2.2
- net N$28: now also VT3.3; no longer VT3.2
- net N$3: now also 2R2.2
- net N$4: now also R14.1; no longer D10.C
- net N$9: now also VT1.2; no longer VT1.3
Routing:
- net N$27: track 5.08 -> 47.1 mm
- net N$26: track 5.08 -> 34.9 mm
- net N$28: track 5.08 -> 21.7 mm
- net +12V: track 10.4 -> 25.1 mm
- net OUT3: track 0.00 -> 14.0 mm
- net GND: track 65.8 -> 78.6 mm
- net OUT2: track 0.00 -> 8.46 mm
- net N$4: track 40.7 -> 33.1 mm, vias 1 -> 0
- net N$23: track 0.00 -> 7.29 mm
- net N$11: track 2.43 -> 6.24 mm
- net +3V3: track 17.8 -> 14.2 mm
- net N$24: track 0.00 -> 3.47 mm
- net N$21: track 5.76 -> 8.33 mm
- net N$25: track 6.79 -> 9.01 mm
- net N$22: track 7.25 -> 9.11 mm
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
Commit message: 8
Parts:
- removed 2R3: 11k, resistor:R0805
- removed 2R4: 18k, resistor:R0805
- removed C15: 100n, resistor:C0805K
- removed D10, D11, D12, D13, D14, D15, D6, D8, D9: (no value), diode:SOD80C
- removed R1, R10, R11, R12, R5, R7, R8, R9: (no value), rcl:R0805
- removed R14, R4, R6: (no value), rcl:R1206W
- added 1R1, 3R1, J1: (no value), rcl:R1206W
- added 1RB, 1RG, 1RR, 2RB, 2RG, 2RR, 3RB, 3RG, 3RR: (no value), rcl:R0805
- added 1VDB, 1VDG, 1VDR, 2VDB, 2VDG, 2VDR, 3VDB, 3VDG, 3VDR: (no value), diode:SOD80C
- added C5: 10m, rcl:C1210
- added R1A: 2r5, resistor:R0805
- 2R1: value 2r5 -> (none); device resistor:R0805 -> rcl:R0805
- C2: value 10m -> 100n; device rcl:C1210 -> resistor:C0805K
- R2: value (none) -> 11k; device rcl:R0805 -> resistor:R0805
- R3: value (none) -> 18k; device rcl:R0805 -> resistor:R0805
- moved R3 48.8 mm to (25.7, 3.81), turned to 0 degrees
- moved R2 44.3 mm to (20.3, 1.59), turned to 90 degrees
- moved 2R1 26.4 mm to (34.6, 14.9), turned to 180 degrees
- moved C1 24.0 mm to (9.53, 11.4), turned to 90 degrees
- moved VT3 7.94 mm to (13.0, 15.6)
- moved C2 3.82 mm to (13.3, 11.1)
- moved VT1 3.49 mm to (19.4, 15.6)
- moved L1 1.62 mm to (25.1, -3.49)
- renumbered 2C1 to C3B, 2C2 to C3A, 2R2 to R1B, C3 to C6, C4 to C7, D1 to VD1
Connections:
- net POWER renamed PWRLED
- net SSD renamed DSKLED
- removed net OUT1: DD1.10, R4.1
- removed net OUT2: DD1.11, DD1.8, R5.1
- removed net OUT3: DD1.13, DD1.4, DD1.9, R6.1
- new net OUT_DSLED: 3R1.1, DD1.13, DD1.4, DD1.9
- new net OUT_PWLED: 2R1.1, DD1.11, DD1.8
- new net OUT_SLED: 1R1.1, DD1.10
- net +12V: now also C1.1, R1A.1; no longer 2R1.1, C15.1
- net +3V3: now also C5.1, R3.2; no longer 2R4.2, C1.1
- net GND: now also C5.2, R2.1; no longer 2R3.1, C15.2
- net N$10: now also 2R1.2; no longer R5.2
- net N$11: now also 2RB.1, 2VDB.A; no longer D10.A, R7.1
- net N$12: now also 1R1.2; no longer R4.2
- net N$13: now also 1VDG.C, 2VDG.C, 3VDG.C; no longer D11.C, D14.C, D8.C
- net N$14: now also 1VDR.C, 2VDR.C, 3VDR.C; no longer D12.C, D15.C, D9.C
- net N$15: now also 2RR.1, 2VDR.A; no longer D12.A, R9.1
- net N$16: now also 2RG.1, 2VDG.A; no longer D11.A, R8.1
- net N$17: now also 3RR.1, 3VDR.A; no longer D15.A, R12.1
- net N$18: now also 3RG.1, 3VDG.A; no longer D14.A, R11.1
- net N$20: now also 3RB.1, 3VDB.A; no longer D13.A, R10.1
- net N$24: now also 2VDB.C, J1.2; no longer D10.C, R14.2
- net N$25: now also R2.2, R3.1; no longer 2R3.2, 2R4.1
- net N$26: now also 3RB.2, 3RG.2, 3RR.2; no longer R10.2, R11.2, R12.2
- net N$27: now also 2RB.2, 2RG.2, 2RR.2; no longer R7.2, R8.2, R9.2
- net N$28: now also 1RB.2, 1RG.2, 1RR.2; no longer R1.2, R2.2, R3.2
- net N$3: now also R1A.2; no longer 2R1.2
- net N$4: now also 1VDB.C, 3VDB.C, J1.1; no longer D13.C, D6.C, R14.1
- net N$6: now also 1RR.1, 1VDR.A; no longer D9.A, R3.1
- net N$7: now also 1RG.1, 1VDG.A; no longer D8.A, R2.1
- net N$8: now also 1RB.1, 1VDB.A; no longer D6.A, R1.1
- net N$9: now also 3R1.2; no longer R6.2
Routing:
- net GND: track 78.6 -> 48.9 mm
- net OUT_DSLED: track 0.00 -> 14.0 mm
- net OUT3: track 14.0 -> 0.00 mm
- net +12V: track 25.1 -> 15.3 mm
- net +3V3: track 14.2 -> 5.04 mm
- net OUT_PWLED: track 0.00 -> 8.46 mm
- net OUT2: track 8.46 -> 0.00 mm
- net N$14: track 44.9 -> 41.8 mm
- net N$16: track 6.24 -> 4.65 mm
- net N$11: track 6.24 -> 4.65 mm
- net N$4: track 33.1 -> 31.6 mm
- net N$27: track 47.1 -> 48.6 mm
- net N$24: track 3.47 -> 2.20 mm

Commit message: 9
Parts:
- moved R1A 42.2 mm to (30.5, -34.6), flipped to the bottom, turned to 90 degrees
- moved R1B 37.1 mm to (26.7, -34.6), flipped to the bottom, turned to 90 degrees
- moved DA1 34.1 mm to (29.2, -29.8), flipped to the bottom, turned to 90 degrees
- moved R2 28.4 mm to (29.2, -25.4), flipped to the bottom, turned to 180 degrees
- moved DD1 25.5 mm to (65.7, 26.4), flipped to the bottom
- moved C3A 24.5 mm to (22.9, -28.6), flipped to the bottom, turned to 90 degrees
- moved R3 24.5 mm to (31.4, -20.0), flipped to the bottom, turned to 90 degrees
- moved VT3 21.6 mm to (-8.26, 12.1)
- moved C3B 21.5 mm to (20.3, -28.6), flipped to the bottom, turned to 90 degrees
- moved VD1 20.1 mm to (23.5, -24.1), flipped to the bottom, turned to 180 degrees
- moved L1 17.2 mm to (24.1, -20.6), flipped to the bottom, turned to 180 degrees
- moved C2 8.13 mm to (19.7, 6.03), flipped to the bottom
- moved C1 7.86 mm to (15.2, 6.03), flipped to the bottom
- moved JP1 7.05 mm to (10.8, 9.21)
- moved JP2 5.43 mm to (1.27, 10.8)
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Routing:
- net GND: track 48.9 -> 17.6 mm
- net N$12: track 0.00 -> 21.4 mm
- net +3V3: track 5.04 -> 20.6 mm
- net N$27: track 48.6 -> 38.9 mm
- net N$21: track 8.33 -> 5.71 mm
- net N$23: track 7.29 -> 9.40 mm
- net N$28: track 21.3 -> 23.1 mm
- net N$4: track 31.6 -> 29.9 mm
- net N$13: track 29.4 -> 30.3 mm
- net N$22: track 9.11 -> 9.83 mm
- net N$16: track 4.65 -> 4.02 mm
- net N$11: track 4.65 -> 4.02 mm
- net N$24: track 2.20 -> 2.83 mm
- net N$26: track 34.5 -> 35.0 mm

Commit message: 11
Parts:
- added +12V: (no value), DSS:CON_PWR_2PIN4MM
- added JP5, JP6: (no value), pinhead:1X01
- 2R1: device rcl:R0805 -> rcl:R1206W
- JP1: device pinhead:1X02 -> pinhead:1X01
- R1B: value 2r5 -> (none)
- moved 2R1 69.2 mm to (-31.4, -5.71), turned to 270 degrees
- moved DD1 61.3 mm to (5.71, 13.7)
- moved 3R1 57.3 mm to (-31.8, 1.91), turned to 180 degrees
- moved VT2 57.2 mm to (-26.0, -7.30), turned to 270 degrees
- moved VT1 47.4 mm to (-26.0, 1.91), turned to 270 degrees
- moved 1R1 46.8 mm to (-31.8, 11.1), turned to 180 degrees
- moved R1A 44.0 mm to (26.4, 9.21), turned to 180 degrees
- moved R1B 41.3 mm to (26.4, 6.67), turned to 180 degrees
- moved C7 31.1 mm to (12.4, 8.57), turned to 180 degrees
- moved DA1 30.5 mm to (24.8, 0.32), turned to 0 degrees
- moved C6 27.8 mm to (11.1, 1.27), turned to 0 degrees
- moved R2 27.2 mm to (20.3, 0.32), turned to 90 degrees
- moved R3 25.5 mm to (16.8, 0.95), turned to 0 degrees
- moved C5 23.7 mm to (12.4, -2.86)
- moved C3A 22.6 mm to (23.5, -6.03), turned to 0 degrees
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Connections:
- net +12V: now also +12V.1; no longer JP1.1
- net +3V3: now also DD1.1, DD1.2
- net DSKLED: now also DD1.8, DD1.9, JP6.1; no longer DD1.5, DD1.6
- net GND: now also +12V.2; no longer JP1.2
- net OUT_DSLED: now also DD1.10, DD1.5; no longer DD1.4, DD1.9
- net OUT_PWLED: now also DD1.6; no longer DD1.8
- net OUT_SLED: now also DD1.4; no longer DD1.10
- net PWRLED: now also JP5.1
Routing:
- net OUT_PWLED: track 8.46 -> 88.6 mm
- net +3V3: track 20.6 -> 87.0 mm
- net OUT_DSLED: track 14.0 -> 66.6 mm
- net GND: track 17.6 -> 66.3 mm
- net OUT_SLED: track 0.00 -> 40.5 mm
- net N$27: track 38.9 -> 9.53 mm
- net N$26: track 35.0 -> 9.53 mm
- net N$12: track 21.4 -> 2.95 mm
- net +12V: track 15.3 -> 31.3 mm
- net N$28: track 23.1 -> 9.53 mm
- net N$21: track 5.71 -> 11.1 mm
- net N$10: track 0.00 -> 4.16 mm
- net PWRLED: track 0.00 -> 3.82 mm
- net DSKLED: track 1.27 -> 5.00 mm
- net N$9: track 0.00 -> 2.95 mm
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Other:
- board size 100 x 33 mm -> 100 x 34.9 mm
