File: pc2_key.brd (EAGLE design)
At the start: 100 x 34.9 mm, 47 parts

Commit message: 12
Parts:
- VT1, VT2, VT3: value KT561 -> KT3107
- renumbered R13 to RC1
Changed lines of the file:
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@@
 <wire x1="-50" y1="-13" x2="50" y2="-13" width="0.254" layer="20"/>
 <wire x1="-50" y1="21.89" x2="50" y2="21.89" width="0.254" layer="20"/>
-<wire x1="-33" y1="19.985" x2="-33" y2="-13" width="0.254" layer="21"/>
-<wire x1="33" y1="19.985" x2="33" y2="-13" width="0.254" layer="22"/>
+<wire x1="-33" y1="21.89" x2="-33" y2="-13" width="0.254" layer="21"/>
+<wire x1="33" y1="21.89" x2="33" y2="-13" width="0.254" layer="21"/>
 </plain>
 <attributes>
@@
 <element name="C2" library="resistor" package="C0805K" value="100n" x="20.6375" y="8.89" rot="MR0"/>
 <element name="DD1" library="40xx" package="SO14" value="4011D" x="5.715" y="13.6525" rot="MR90"/>
-<element name="VT1" library="m_transistor" package="TO92" value="KT561" x="-26.035" y="1.905" rot="R270"/>
-<element name="VT2" library="m_transistor" package="TO92" value="KT561" x="-26.035" y="-7.3025" rot="R270"/>
-<element name="VT3" library="m_transistor" package="TO92" value="KT561" x="-26.035" y="11.1125" rot="R270"/>
+<element name="VT1" library="m_transistor" package="TO92" value="KT3107" x="-26.035" y="1.905" rot="R270"/>
+<element name="VT2" library="m_transistor" package="TO92" value="KT3107" x="-26.035" y="-7.3025" rot="R270"/>
+<element name="VT3" library="m_transistor" package="TO92" value="KT3107" x="-26.035" y="11.1125" rot="R270"/>
 <element name="1RB" library="rcl" package="R0805" value="" x="-21.9075" y="11.7475" smashed="yes" rot="MR0">
 <attribute name="NAME" x="-24.13" y="11.1125" size="1.27" layer="26" rot="MR0"/>
@@
 <element name="JP2" library="pinhead" package="1X02" value="" x="-5.715" y="10.4775" rot="R180"/>
 <element name="C3B" library="resistor" package="C0805K" value="59" x="23.495" y="-8.5725" rot="MR0"/>
-<element name="R13" library="rcl" package="R0805" value="10" x="7.3025" y="-4.7625" rot="MR90"/>
+<element name="RC1" library="rcl" package="R0805" value="10" x="7.3025" y="-4.7625" rot="MR90"/>
 <element name="J1" library="rcl" package="R1206W" value="" x="-9.2075" y="-4.7625" smashed="yes" rot="MR0">
 <attribute name="NAME" x="-7.3025" y="-6.0325" size="1.27" layer="26" rot="MR180"/>
@@
 <wire x1="20.32" y1="-3.1975" x2="19.05" y2="-3.1975" width="0.6096" layer="16"/>
 <wire x1="20.32" y1="-0.5325" x2="20.32" y2="-3.1975" width="0.6096" layer="16"/>
-<contactref element="R13" pad="1"/>
+<contactref element="RC1" pad="1"/>
 <wire x1="16.51" y1="20.6375" x2="16.8275" y2="20.6375" width="0.6096" layer="16"/>
 <wire x1="16.8275" y1="8.5725" x2="13.3825" y2="8.5725" width="1.27" layer="16"/>
@@
 <signal name="N$23">
 <contactref element="S1" pad="D3"/>
-<contactref element="R13" pad="2"/>
+<contactref element="RC1" pad="2"/>
 <wire x1="1.27" y1="-5.08" x2="1.27" y2="-2.8575" width="0.6096" layer="16"/>
 <wire x1="1.27" y1="-2.8575" x2="2.54" y2="-1.5875" width="0.6096" layer="16"/>

Commit message: 14
Parts:
- removed JP1: (no value), pinhead:1X01
- added R1: (no value), rcl:M0805
- added R4: (no value), rcl:R1206W
- R1A, R1B: device resistor:R0805 -> resistor:R1206
- moved C1 10.4 mm to (19.7, 8.89)
- moved C6 4.55 mm to (9.21, -2.86), turned to 270 degrees
- moved C2 3.24 mm to (21.3, 5.71)
- moved RC1 2.73 mm to (8.89, -6.99), turned to 0 degrees
- moved R3 1.90 mm to (16.8, 2.86)
- moved C3B 0.95 mm to (23.5, -7.62)
- moved L1 0.63 mm to (15.6, -4.13)
- moved C5 0.32 mm to (12.1, -2.86)
- moved C3A 0.32 mm to (23.5, -5.71)
- moved DD1 0.32 mm to (5.40, 13.7)
- turned HDDLED to 0 degrees
- turned PWRLED to 180 degrees
- renumbered JP5 to PWRLED, JP6 to HDDLED
Connections:
- net DSKLED: now also R4.2
- net GND: now also R1.1, R4.1
- net PWRLED: now also R1.2
Routing:
- net GND: track 66.3 -> 132.4 mm
- net +3V3: track 87.0 -> 104.0 mm
- net +12V: track 31.3 -> 18.0 mm
- net N$23: track 9.40 -> 12.8 mm
- net DSKLED: track 5.00 -> 7.83 mm
- net OUT_PWLED: track 88.6 -> 91.4 mm
- net PWRLED: track 3.82 -> 6.36 mm
- net N$5: track 6.44 -> 5.66 mm

Commit message: 15
Parts:
- added C3: 10m, rcl:C1210
- added L2: (no value), rcl:L1812
- moved C6 4.85 mm to (11.7, 1.27), turned to 0 degrees
- moved R3 1.71 mm to (16.2, 1.27)
Connections:
- net +12V renamed N$30
- new net N$29: C5.1, C6.1, L1.2, L2.1, R3.2
- net +3V3: now also C3.1, L2.2; no longer C5.1, C6.1, L1.2, R3.2
- net GND: now also C3.2
Routing:
- net +3V3: track 104.0 -> 88.8 mm
- net N$29: track 0.00 -> 13.4 mm
- net GND: track 132.4 -> 141.2 mm
- net N$25: track 7.15 -> 8.70 mm
Changed lines of the file:
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@@
 <element name="R1A" library="resistor" package="R1206" value="2r5" x="26.3525" y="9.2075" rot="MR180"/>
 <element name="R2" library="resistor" package="R0805" value="11k" x="20.32" y="0.3175" rot="MR90"/>
-<element name="R3" library="resistor" package="R0805" value="18k" x="16.8275" y="2.8575" rot="MR0"/>
+<element name="R3" library="resistor" package="R0805" value="18k" x="16.1925" y="1.27" rot="MR0"/>
 <element name="C2" library="resistor" package="C0805K" value="100n" x="21.2725" y="5.715" rot="MR0"/>
 <element name="DD1" library="40xx" package="SO14" value="4011D" x="5.3975" y="13.6525" rot="MR90"/>
@@
 <element name="C5" library="rcl" package="C1210" value="10m" x="12.065" y="-2.8575" rot="MR270"/>
 <element name="C1" library="rcl" package="C1210" value="10m" x="19.685" y="8.89" rot="MR0"/>
-<element name="C6" library="resistor" package="C0805K" value="100n" x="9.2075" y="-2.8575" rot="MR270"/>
+<element name="C6" library="resistor" package="C0805K" value="100n" x="11.7475" y="1.27" rot="MR0"/>
 <element name="C7" library="resistor" package="C0805K" value="100n" x="12.3825" y="8.5725" rot="MR180"/>
 <element name="JP2" library="pinhead" package="1X02" value="" x="-5.715" y="10.4775" rot="R180"/>
@@
 <element name="R1" library="rcl" package="M0805" value="" x="15.5575" y="11.43" rot="MR0"/>
 <element name="R4" library="rcl" package="R1206W" value="" x="15.875" y="15.24" rot="MR0"/>
+<element name="L2" library="rcl" package="L1812" value="" x="14.2875" y="5.08" rot="MR0"/>
+<element name="C3" library="rcl" package="C1210" value="10m" x="7.9375" y="4.1275" rot="MR270"/>
 </elements>
 <signals>
@@
 <wire x1="12.065" y1="-6.985" x2="12.065" y2="-10.16" width="1.27" layer="16"/>
 <wire x1="9.84" y1="-6.985" x2="12.065" y2="-6.985" width="1.27" layer="16"/>
-<wire x1="9.2075" y1="-3.8575" x2="9.6075" y2="-4.2575" width="1.016" layer="16"/>
 <wire x1="9.6075" y1="-4.2575" x2="12.065" y2="-4.2575" width="1.016" layer="16"/>
 <contactref element="R1" pad="1"/>
@@
 <wire x1="17.374" y1="15.24" x2="17.4625" y2="15.24" width="0.6096" layer="16"/>
 <wire x1="16.5075" y1="11.43" x2="17.4625" y2="11.43" width="0.6096" layer="16"/>
+<contactref element="C3" pad="2"/>
+<wire x1="9.6075" y1="-4.2575" x2="8.89" y2="-3.54" width="1.016" layer="16"/>
+<wire x1="8.89" y1="-3.54" x2="8.89" y2="1.27" width="1.016" layer="16"/>
+<wire x1="8.89" y1="1.27" x2="10.7475" y2="1.27" width="1.016" layer="16"/>
+<wire x1="7.9375" y1="2.7275" x2="8.89" y2="1.27" width="1.016" layer="16"/>
 </signal>
 <signal name="N$25">
@@
 <wire x1="20.32" y1="2.9175" x2="20.32" y2="1.1675" width="0.6096" layer="16"/>
 <wire x1="20.32" y1="0.9525" x2="20.32" y2="1.1675" width="0.6096" layer="16"/>
-<wire x1="17.6775" y1="2.8575" x2="18.055" y2="2.9175" width="0.6096" layer="16"/>
+<wire x1="17.0425" y1="1.27" x2="18.055" y2="2.9175" width="0.6096" layer="16"/>
 <wire x1="18.055" y1="2.9175" x2="20.32" y2="2.9175" width="0.6096" layer="16"/>
 </signal>
@@
 <contactref element="VT2" pad="1"/>
 <contactref element="VT1" pad="1"/>
-<contactref element="R3" pad="2"/>
-<contactref element="L1" pad="2"/>
-<contactref element="C5" pad="1"/>
-<contactref element="C6" pad="1"/>
 <contactref element="C7" pad="1"/>
 <contactref element="DD1" pad="14"/>
@@
 <wire x1="2.3241" y1="11.1125" x2="2.3241" y2="9.8425" width="0.6096" layer="16"/>
 <wire x1="2.3241" y1="9.8425" x2="8.4709" y2="9.8425" width="0.6096" layer="16"/>
-<wire x1="8.7884" y1="8.5725" x2="-0.635" y2="8.5725" width="0.6096" layer="16"/>
+<wire x1="8.4709" y1="8.5725" x2="-0.635" y2="8.5725" width="0.6096" layer="16"/>
 <wire x1="-1.5875" y1="11.7475" x2="-4.1275" y2="14.2875" width="0.6096" layer="16"/>
 <wire x1="-4.1275" y1="14.2875" x2="-24.13" y2="14.2875" width="0.6096" layer="16"/>
 <wire x1="-24.13" y1="14.2875" x2="-24.765" y2="13.6525" width="0.6096" layer="16"/>
 <wire x1="-24.765" y1="13.6525" x2="-27.305" y2="13.6525" width="0.6096" layer="16"/>
-<wire x1="8.4709" y1="9.8425" x2="8.7884" y2="8.5725" width="0.6096" layer="16"/>
-<wire x1="8.7884" y1="8.5725" x2="11.3825" y2="8.5725" width="0.6096" layer="16"/>
+<wire x1="8.4709" y1="9.8425" x2="8.4709" y2="8.5725" width="0.6096" layer="16"/>
+<wire x1="8.4709" y1="8.5725" x2="11.3825" y2="8.5725" width="0.6096" layer="16"/>
 <wire x1="-1.5875" y1="11.7475" x2="-1.5875" y2="9.525" width="0.6096" layer="16"/>
 <wire x1="-1.5875" y1="9.525" x2="-0.635" y2="8.5725" width="0.6096" layer="16"/>
-<wire x1="15.5575" y1="-1.6275" x2="15.3875" y2="-1.4575" width="1.27" layer="16"/>
-<wire x1="15.3875" y1="-1.4575" x2="12.065" y2="-1.4575" width="1.27" layer="16"/>
-<wire x1="9.2075" y1="-1.8575" x2="9.2075" y2="-1.905" width="1.016" layer="16"/>
-<wire x1="9.2075" y1="-1.8575" x2="9.2075" y2="-1.4575" width="1.016" layer="16"/>
-<wire x1="9.2075" y1="-1.4575" x2="12.065" y2="-1.4575" width="1.016" layer="16"/>
-<wire x1="9.2075" y1="0.5425" x2="9.2075" y2="-1.8575" width="1.016" layer="16"/>
-<wire x1="15.9775" y1="2.8575" x2="11.43" y2="2.8575" width="1.016" layer="16"/>
-<wire x1="11.43" y1="2.8575" x2="11.3825" y2="2.8575" width="1.016" layer="16"/>
-<wire x1="11.3825" y1="2.8575" x2="11.3825" y2="8.5725" width="1.016" layer="16"/>
-<wire x1="9.2075" y1="0.5425" x2="11.43" y2="2.765" width="1.016" layer="16"/>
-<wire x1="11.43" y1="2.765" x2="11.43" y2="2.8575" width="1.016" layer="16"/>
+<contactref element="L2" pad="2"/>
+<contactref element="C3" pad="1"/>
+<wire x1="12.3375" y1="5.08" x2="9.0775" y2="5.08" width="0.6096" layer="16"/>
+<wire x1="9.0775" y1="5.08" x2="7.9375" y2="5.5275" width="0.6096" layer="16"/>
+<wire x1="8.4709" y1="8.5725" x2="8.4709" y2="6.2641" width="1.016" layer="16"/>
+<wire x1="8.4709" y1="6.2641" x2="7.9375" y2="5.5275" width="1.016" layer="16"/>
 </signal>
 <signal name="N$9">
@@
 <wire x1="19.685" y1="-10.16" x2="19.05" y2="-9.525" width="1.016" layer="16"/>
 <wire x1="19.05" y1="-9.525" x2="19.05" y2="-7.5975" width="1.016" layer="16"/>
-</signal>
-<signal name="+12V">
-<contactref element="DA1" pad="6"/>
-<contactref element="R1A" pad="1"/>
-<contactref element="C2" pad="1"/>
-<contactref element="C1" pad="1"/>
-<contactref element="R1B" pad="1"/>
-<contactref element="+12V" pad="1"/>
-<wire x1="24.13" y1="2.9175" x2="24.13" y2="5.715" width="0.6096" layer="16"/>
-<wire x1="22.2725" y1="5.715" x2="24.13" y2="5.715" width="0.6096" layer="16"/>
-<wire x1="24.13" y1="5.715" x2="24.9305" y2="6.6675" width="0.6096" layer="16"/>
-<wire x1="21.085" y1="8.89" x2="25.185" y2="8.89" width="0.6096" layer="16"/>
-<wire x1="25.185" y1="8.89" x2="24.9305" y2="9.2075" width="0.6096" layer="16"/>
-<wire x1="24.9305" y1="9.2075" x2="24.9305" y2="6.6675" width="1.016" layer="16"/>
-<wire x1="24.9305" y1="9.2075" x2="24.9305" y2="13.2645" width="1.016" layer="16"/>
-<wire x1="24.9305" y1="13.2645" x2="24.225" y2="13.97" width="1.016" layer="16"/>
 </signal>
 <signal name="N$21">
@@
 <wire x1="-13.54" y1="-4.7625" x2="-10.7065" y2="-4.7625" width="0.6096" layer="16"/>
 </signal>
+<signal name="N$29">
+<contactref element="R3" pad="2"/>
+<contactref element="L1" pad="2"/>
+<contactref element="C5" pad="1"/>
+<contactref element="C6" pad="1"/>
+<contactref element="L2" pad="1"/>
+<wire x1="15.5575" y1="-1.6275" x2="15.3875" y2="-1.4575" width="1.27" layer="16"/>
+<wire x1="15.3875" y1="-1.4575" x2="13.0175" y2="-1.4575" width="1.27" layer="16"/>
+<wire x1="13.0175" y1="-1.4575" x2="12.065" y2="-1.4575" width="1.27" layer="16"/>
+<wire x1="15.3425" y1="1.27" x2="15.3425" y2="-1.4125" width="1.016" layer="16"/>
+<wire x1="15.3425" y1="-1.4125" x2="15.5575" y2="-1.6275" width="1.016" layer="16"/>
+<wire x1="15.3425" y1="1.27" x2="15.3425" y2="3.2325" width="1.016" layer="16"/>
+<wire x1="15.3425" y1="3.2325" x2="16.2375" y2="5.08" width="1.016" layer="16"/>
+<wire x1="12.7475" y1="1.27" x2="12.7475" y2="-1.1875" width="1.016" layer="16"/>
+<wire x1="12.7475" y1="-1.1875" x2="13.0175" y2="-1.4575" width="1.016" layer="16"/>
+</signal>
+<signal name="N$30">
+<contactref element="DA1" pad="6"/>
+<contactref element="R1A" pad="1"/>
+<contactref element="C2" pad="1"/>
+<contactref element="C1" pad="1"/>
+<contactref element="R1B" pad="1"/>
+<contactref element="+12V" pad="1"/>
+<wire x1="24.13" y1="2.9175" x2="24.13" y2="5.715" width="0.6096" layer="16"/>
+<wire x1="22.2725" y1="5.715" x2="24.13" y2="5.715" width="0.6096" layer="16"/>
+<wire x1="24.13" y1="5.715" x2="24.9305" y2="6.6675" width="0.6096" layer="16"/>
+<wire x1="21.085" y1="8.89" x2="25.185" y2="8.89" width="0.6096" layer="16"/>
+<wire x1="25.185" y1="8.89" x2="24.9305" y2="9.2075" width="0.6096" layer="16"/>
+<wire x1="24.9305" y1="9.2075" x2="24.9305" y2="6.6675" width="1.016" layer="16"/>
+<wire x1="24.9305" y1="9.2075" x2="24.9305" y2="13.2645" width="1.016" layer="16"/>
+<wire x1="24.9305" y1="13.2645" x2="24.225" y2="13.97" width="1.016" layer="16"/>
+</signal>
 </signals>
