File: pc2_key.brd (EAGLE design)
At the start: 100 x 34.9 mm, 50 parts

Commit message: 17
Parts:
- added GND: (no value), pinhead:1X01
- moved JP2 1.35 mm to (-4.76, 9.53)
- moved HDDLED 0.95 mm to (12.4, 15.6)
- moved PWRLED 0.95 mm to (12.4, 10.5)
- moved R1 0.95 mm to (15.6, 10.5)
- moved R4 0.95 mm to (15.9, 14.3)
- moved L2 0.90 mm to (13.7, 4.45)
- moved 1VDR 0.64 mm to (-16.8, 6.03)
- moved C7 0.63 mm to (12.4, 7.94)
Connections:
- net GND: now also GND.1
Routing:
- net N$21: track 11.1 -> 8.80 mm
- net N$22: track 9.25 -> 7.59 mm
- net OUT_PWLED: track 91.4 -> 92.8 mm
- net N$29: track 13.4 -> 12.6 mm
- net N$4: track 29.9 -> 29.2 mm
- net +3V3: track 88.8 -> 88.2 mm
- net N$7: track 11.8 -> 11.2 mm
- net N$14: track 42.3 -> 41.8 mm

Commit message: 18
Parts:
- L1: device rcl:6000-XXXX-RC -> inductor-neosid:SD12K100
- moved VD1 0.95 mm to (20.0, -5.40)
- moved L1 0.63 mm to (16.2, -4.13)
- moved C3A 0.45 mm to (23.8, -6.03)
- moved C3B 0.45 mm to (23.8, -7.94)
- moved C5 0.32 mm to (11.7, -2.86)
- renumbered JP2 to SW1
Routing:
- net N$29: track 12.6 -> 14.1 mm

Commit message: 18
Parts:
- added 3VDB1: LL4148, diode:SOD80C
- added F1: (no value), fuse:SH32
- added J2: (no value), rcl:R1206W
- added SJ1: (no value), jumper:SJ
- added U$5, U$6, U$7, U$8: (no value), marks:ANGLE-SW-1
- C3, C5: value 10m -> 22m
- L1: device inductor-neosid:SD12K100 -> ct-pack:LH7X10MM
- L2: value (none) -> 10mkhn; device rcl:L1812 -> rcl:PIS2816
- moved J1 21.8 mm to (8.26, 8.26)
- moved R1A 15.3 mm to (32.7, -4.76), turned to 0 degrees
- moved R1B 15.3 mm to (32.7, -7.30), turned to 0 degrees
- moved L1 5.28 mm to (21.3, -5.56), flipped to the top, turned to 270 degrees
- moved R3 5.26 mm to (21.0, 3.49)
- moved C6 3.88 mm to (9.53, -1.91)
- moved C5 3.24 mm to (11.1, -6.03)
- moved RC1 2.84 mm to (7.62, -9.53)
- moved L2 1.85 mm to (14.6, 2.86), turned to 90 degrees
- moved C7 1.27 mm to (13.7, 7.94)
- moved R2 0.95 mm to (21.3, 0.32)
- moved C3A 0.64 mm to (24.4, -6.03)
- moved C3B 0.64 mm to (24.4, -7.94)
- moved SW1 0.63 mm to (-5.40, 9.53)
- moved DA1 0.63 mm to (25.4, 0.32)
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Connections:
- new net N$32: 3VDB1.C, DD1.3
- new net N$33: +12V.1, F1.P$1
- new net N$34: DD1.1, DD1.2, J1.2
- net +3V3: no longer DD1.1, DD1.2
- net GND: now also SJ1.1
- net N$19: now also L1.2; no longer L1.1
- net N$21: now also 3VDB1.A, SJ1.2
- net N$24: now also J2.2; no longer J1.2
- net N$29: now also L1.1; no longer L1.2
- net N$30: now also F1.P$2; no longer +12V.1
- net N$4: now also J2.1; no longer J1.1
- net PWRLED: now also J1.1
Routing:
- net GND: track 141.0 -> 173.0 mm
- net N$30: track 18.0 -> 32.7 mm
- net N$33: track 0.00 -> 10.2 mm
- net N$34: track 0.00 -> 6.36 mm
- net N$32: track 0.00 -> 4.70 mm
- net N$29: track 14.1 -> 18.5 mm
- net N$25: track 8.70 -> 4.78 mm
- net +3V3: track 88.2 -> 84.6 mm
- net PWRLED: track 6.84 -> 10.4 mm
- net N$21: track 8.80 -> 12.3 mm
- net N$23: track 12.6 -> 14.7 mm
- net N$3: track 13.3 -> 14.2 mm
- added copper zone on layer 16, net N$19
- added copper zone on layer 16, net N$29
Other:
- board size 100 x 34.9 mm -> 98 x 35 mm

Commit message: 19
Parts:
- removed R1: (no value), rcl:M0805
- added R5: 10k, rcl:R1206W
- C3A: value 59 -> 68
- C3B: value 59 -> (none)
- J1, J2: value (none) -> 0
- R1A: value 2r5 -> 4R7
- R1B: value (none) -> 4R7
- R2: value 11k -> 8k2
- R3: value 18k -> 15k
- R4: value (none) -> 10k; device rcl:R1206W -> rcl:M0805
- moved R4 3.82 mm to (15.6, 10.5)
- renumbered C3 to C8
Connections:
- net +3V3 renamed VCC
- net N$25 renamed 1,25V
- net N$29 renamed 3V5
- net DSKLED: now also R5.2; no longer R4.2
- net GND: now also R5.1; no longer R1.1
- net PWRLED: now also R4.2; no longer R1.2
Routing:
- added copper zone on layer 16, net GND
- added copper zone on layer 16, net N$33

Commit message: 20
Parts:
- removed 3VDB1: LL4148, diode:SOD80C
- removed J1: 0, rcl:R1206W
- removed SJ1: (no value), jumper:SJ
- C1: value 10m -> 33m
- RC1: value 10 -> 22
- moved DD1 0.63 mm to (5.40, 14.3)
- renumbered HDDLED to !HDDLED
Connections:
- net DSKLED renamed !DSKLED
- net OUT_PWLED renamed !OUT_PWLED
- net OUT_SLED renamed !OUT_SLED
- removed net N$32: 3VDB1.C, DD1.3
- removed net N$34: DD1.1, DD1.2, J1.2
- removed net OUT_DSLED: 3R1.1, DD1.10, DD1.13, DD1.5
- new net !OUT_DSLED: 3R1.1, DD1.13, DD1.3, DD1.5
- new net N$29: DD1.1, DD1.10, DD1.2
- net GND: no longer SJ1.1
- net N$21: no longer 3VDB1.A, SJ1.2
- net PWRLED: no longer J1.1
Routing:
- net !OUT_DSLED: track 0.00 -> 75.0 mm
- net OUT_DSLED: track 66.2 -> 0.00 mm
- net N$29: track 0.00 -> 9.74 mm
- net N$34: track 6.36 -> 0.00 mm
- net N$32: track 4.70 -> 0.00 mm
- net PWRLED: track 10.4 -> 7.19 mm
- net GND: track 173.3 -> 170.3 mm
- net N$21: track 12.3 -> 9.35 mm

Commit message: .
Parts:
- 1R1, 2R1, 3R1: value (none) -> 5k1
- 1RB: value (none) -> 47k&330k
- 1RG: value (none) -> 20k&120k
- 1RR: value (none) -> 470
- 2RB: value (none) -> 2k7&15k
- 2RG: value (none) -> 3k3
- 2RR: value (none) -> 3k8&150
- VT1, VT2, VT3: value KT3107 -> KT3107Ж
Connections:
- net 3V5 renamed 3V6
- net N$13 renamed G
- net N$14 renamed R
- net N$4 renamed B
Other:
- board text added: "POWER"
- board text added: "STAND"
Changed lines of the file:
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@@
 <wire x1="-50" y1="-13" x2="-50" y2="22" width="0.1524" layer="20"/>
 <dimension x1="77.305" y1="12.8725" x2="69.94" y2="13.1425" x3="73.6225" y3="18.6175" textsize="1.778" layer="47" dtype="horizontal"/>
+<text x="-24.13" y="16.51" size="1.778" layer="22" rot="MR0">STAND</text>
+<text x="-34.29" y="-7.3025" size="1.778" layer="22" rot="MR0">POWER</text>
 </plain>
 <attributes>
@@
 <element name="C2" library="resistor" package="C0805K" value="100n" x="21.2725" y="5.715" rot="MR0"/>
 <element name="DD1" library="40xx" package="SO14" value="4011D" x="5.3975" y="14.2875" rot="MR90"/>
-<element name="VT1" library="m_transistor" package="TO92" value="KT3107" x="-26.035" y="1.905" smashed="yes" rot="R270">
+<element name="VT1" library="m_transistor" package="TO92" value="KT3107Ж" x="-26.035" y="1.905" smashed="yes" rot="R270">
 <attribute name="NAME" x="-32.512" y="3.81" size="1.27" layer="25" ratio="10" rot="R270"/>
 <attribute name="VALUE" x="-30.607" y="5.08" size="1.27" layer="27" ratio="10" rot="R270"/>
 </element>
-<element name="VT2" library="m_transistor" package="TO92" value="KT3107" x="-26.035" y="-7.3025" smashed="yes" rot="R270">
+<element name="VT2" library="m_transistor" package="TO92" value="KT3107Ж" x="-26.035" y="-7.3025" smashed="yes" rot="R270">
 <attribute name="NAME" x="-32.512" y="-5.715" size="1.27" layer="25" ratio="10" rot="R270"/>
 <attribute name="VALUE" x="-30.607" y="-4.1275" size="1.27" layer="27" ratio="10" rot="R270"/>
 </element>
-<element name="VT3" library="m_transistor" package="TO92" value="KT3107" x="-26.035" y="11.1125" smashed="yes" rot="R270">
+<element name="VT3" library="m_transistor" package="TO92" value="KT3107Ж" x="-26.035" y="11.1125" smashed="yes" rot="R270">
 <attribute name="NAME" x="-32.512" y="12.3825" size="1.27" layer="25" ratio="10" rot="R270"/>
 <attribute name="VALUE" x="-30.607" y="14.2875" size="1.27" layer="27" ratio="10" rot="R270"/>
 </element>
-<element name="1RB" library="rcl" package="R0805" value="" x="-21.9075" y="11.7475" smashed="yes" rot="MR0">
+<element name="1RB" library="rcl" package="R0805" value="47k&amp;330k" x="-21.9075" y="11.7475" smashed="yes" rot="MR0">
 <attribute name="NAME" x="-20.13" y="13.1125" size="1.27" layer="26" rot="MR0"/>
 <attribute name="VALUE" x="-21.2725" y="9.2075" size="1.27" layer="28" rot="MR0"/>
 </element>
-<element name="1RG" library="rcl" package="R0805" value="" x="-21.9075" y="9.2075" smashed="yes" rot="MR0">
+<element name="1RG" library="rcl" package="R0805" value="20k&amp;120k" x="-21.9075" y="9.2075" smashed="yes" rot="MR0">
 <attribute name="NAME" x="-30.1625" y="7.9375" size="1.27" layer="26" rot="MR0"/>
 <attribute name="VALUE" x="-21.2725" y="6.6675" size="1.27" layer="28" rot="MR0"/>
 </element>
-<element name="1RR" library="rcl" package="R0805" value="" x="-21.9075" y="6.6675" smashed="yes" rot="MR0">
+<element name="1RR" library="rcl" package="R0805" value="470" x="-21.9075" y="6.6675" smashed="yes" rot="MR0">
 <attribute name="NAME" x="-30.0825" y="6.0325" size="1.27" layer="26" rot="MR0"/>
 <attribute name="VALUE" x="-21.2725" y="4.1275" size="1.27" layer="28" rot="MR0"/>
 </element>
-<element name="1R1" library="rcl" package="R1206W" value="" x="-31.75" y="11.1125" smashed="yes" rot="MR180">
+<element name="1R1" library="rcl" package="R1206W" value="5k1" x="-31.75" y="11.1125" smashed="yes" rot="MR180">
 <attribute name="NAME" x="-34.925" y="10.4775" size="1.27" layer="26" rot="MR0"/>
 <attribute name="VALUE" x="-33.655" y="13.6525" size="1.27" layer="28" rot="MR180"/>
 </element>
-<element name="2R1" library="rcl" package="R1206W" value="" x="-31.4325" y="-5.715" smashed="yes" rot="MR270">
+<element name="2R1" library="rcl" package="R1206W" value="5k1" x="-31.4325" y="-5.715" smashed="yes" rot="MR270">
 <attribute name="NAME" x="-30.7975" y="-8.255" size="1.27" layer="26" rot="MR270"/>
 <attribute name="VALUE" x="-28.8925" y="-3.81" size="1.27" layer="28" rot="MR270"/>
 </element>
-<element name="3R1" library="rcl" package="R1206W" value="" x="-31.75" y="1.905" smashed="yes" rot="MR180">
+<element name="3R1" library="rcl" package="R1206W" value="5k1" x="-31.75" y="1.905" smashed="yes" rot="MR180">
 <attribute name="NAME" x="-34.925" y="1.27" size="1.27" layer="26" rot="MR0"/>
 <attribute name="VALUE" x="-33.655" y="4.445" size="1.27" layer="28" rot="MR180"/>
@@
 <attribute name="VALUE" x="-15.3035" y="3.6195" size="1.27" layer="28" rot="MR0"/>
 </element>
-<element name="2RB" library="rcl" package="R0805" value="" x="-21.9075" y="-4.7625" smashed="yes" rot="MR0">
+<element name="2RB" library="rcl" package="R0805" value="2k7&amp;15k" x="-21.9075" y="-4.7625" smashed="yes" rot="MR0">
 <attribute name="NAME" x="-33.3375" y="-4.7625" size="1.27" layer="26" rot="MR0"/>
 <attribute name="VALUE" x="-21.2725" y="-7.3025" size="1.27" layer="28" rot="MR0"/>
 </element>
-<element name="2RG" library="rcl" package="R0805" value="" x="-21.9075" y="-7.3025" smashed="yes" rot="MR0">
-<attribute name="NAME" x="-33.3375" y="-7.9375" size="1.27" layer="26" rot="MR0"/>
+<element name="2RG" library="rcl" package="R0805" value="3k3" x="-21.9075" y="-7.3025" smashed="yes" rot="MR0">
+<attribute name="NAME" x="-33.3375" y="-9.525" size="1.27" layer="26" rot="MR0"/>
 <attribute name="VALUE" x="-21.2725" y="-9.8425" size="1.27" layer="28" rot="MR0"/>
 </element>
-<element name="2RR" library="rcl" package="R0805" value="" x="-21.9075" y="-9.8425" smashed="yes" rot="MR0">
-<attribute name="NAME" x="-33.3375" y="-10.4775" size="1.27" layer="26" rot="MR0"/>
+<element name="2RR" library="rcl" package="R0805" value="3k8&amp;150" x="-21.9075" y="-9.8425" smashed="yes" rot="MR0">
+<attribute name="NAME" x="-33.3375" y="-11.43" size="1.27" layer="26" rot="MR0"/>
 <attribute name="VALUE" x="-21.2725" y="-12.3825" size="1.27" layer="28" rot="MR0"/>
 </element>
@@
 <wire x1="-30.251" y1="11.1125" x2="-27.305" y2="11.1125" width="0.6096" layer="16"/>
 </signal>
-<signal name="N$4">
+<signal name="B">
 <contactref element="S1" pad="D1"/>
 <contactref element="3VDB" pad="C"/>
@@
 <wire x1="-4.1275" y1="-4.7625" x2="-3.81" y2="-5.08" width="0.6096" layer="16"/>
 </signal>
-<signal name="N$13">
+<signal name="G">
 <contactref element="S1" pad="D2"/>
 <contactref element="2VDG" pad="C"/>
@@
 <wire x1="-12.065" y1="-0.205" x2="-12.065" y2="1.7925" width="0.6096" layer="16"/>
 </signal>
-<signal name="N$14">
+<signal name="R">
 <contactref element="S1" pad="D4"/>
 <contactref element="3VDR" pad="C"/>
@@
 <wire x1="-13.54" y1="-4.7625" x2="-10.7065" y2="-4.7625" width="0.6096" layer="16"/>
 </signal>
-<signal name="3V5">
+<signal name="3V6">
 <contactref element="R3" pad="2"/>
 <contactref element="L1" pad="1"/>

Commit message: .
Parts:
- 3RB: value (none) -> 9k1&200k
- 3RG: value (none) -> 20k&27k
- 3RR: value (none) -> 1k&1k
Changed lines of the file:
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@@
 <attribute name="VALUE" x="-15.3035" y="-12.2555" size="1.27" layer="28" rot="MR0"/>
 </element>
-<element name="3RB" library="rcl" package="R0805" value="" x="-21.9075" y="3.4925" smashed="yes" rot="MR0">
+<element name="3RB" library="rcl" package="R0805" value="9k1&amp;200k" x="-21.9075" y="3.4925" smashed="yes" rot="MR0">
 <attribute name="NAME" x="-30.1625" y="3.4925" size="1.27" layer="26" rot="MR0"/>
 <attribute name="VALUE" x="-21.2725" y="0.9525" size="1.27" layer="28" rot="MR0"/>
 </element>
-<element name="3RG" library="rcl" package="R0805" value="" x="-21.9075" y="0.9525" smashed="yes" rot="MR0">
+<element name="3RG" library="rcl" package="R0805" value="20k&amp;27k" x="-21.9075" y="0.9525" smashed="yes" rot="MR0">
 <attribute name="NAME" x="-30.1625" y="-0.9525" size="1.27" layer="26" rot="MR0"/>
 <attribute name="VALUE" x="-21.2725" y="-1.5875" size="1.27" layer="28" rot="MR0"/>
 </element>
-<element name="3RR" library="rcl" package="R0805" value="" x="-21.9075" y="-1.5875" smashed="yes" rot="MR0">
+<element name="3RR" library="rcl" package="R0805" value="1k&amp;1k" x="-21.9075" y="-1.5875" smashed="yes" rot="MR0">
 <attribute name="NAME" x="-30.1625" y="-2.8575" size="1.27" layer="26" rot="MR0"/>
 <attribute name="VALUE" x="-21.2725" y="-4.1275" size="1.27" layer="28" rot="MR0"/>
@@
 <wire x1="-22.8575" y1="-0.635" x2="-22.8575" y2="0.9525" width="0.6096" layer="16"/>
 <wire x1="-22.8575" y1="0.9525" x2="-22.8575" y2="3.4925" width="0.6096" layer="16"/>
-<wire x1="-27.305" y1="-0.635" x2="-22.8575" y2="-0.635" width="0.6096" layer="16"/>
+<wire x1="-27.305" y1="-0.635" x2="-22.8575" y2="-0.635" width="1.016" layer="16"/>
 </signal>
 <signal name="N$27">
@@
 <wire x1="-22.8575" y1="-9.8425" x2="-22.8575" y2="-7.3025" width="0.6096" layer="16"/>
 <wire x1="-22.8575" y1="-7.3025" x2="-22.8575" y2="-4.7625" width="0.6096" layer="16"/>
-<wire x1="-27.305" y1="-9.8425" x2="-22.8575" y2="-9.8425" width="0.6096" layer="16"/>
+<wire x1="-27.305" y1="-9.8425" x2="-22.8575" y2="-9.8425" width="1.016" layer="16"/>
 </signal>
 <signal name="N$28">
@@
 <wire x1="-22.8575" y1="8.5725" x2="-22.8575" y2="9.2075" width="0.6096" layer="16"/>
 <wire x1="-22.8575" y1="9.2075" x2="-22.8575" y2="11.7475" width="0.6096" layer="16"/>
-<wire x1="-27.305" y1="8.5725" x2="-22.8575" y2="8.5725" width="0.6096" layer="16"/>
+<wire x1="-27.305" y1="8.5725" x2="-22.8575" y2="8.5725" width="1.016" layer="16"/>
 </signal>
 <signal name="N$3">
