File: pc2_key.sch (EAGLE design)
At the start: 25 parts, among them IC1 4011D, IC2 MC34063AD

Commit message: 2
Parts:
- removed 1C10: 220u/6V, resistor:CPOL-EUE3.5-8
- removed 1R15: 27K, resistor:R-EU_R0805
- removed 2D1: 1N5819, diode:DIODE-DO41-10
- removed 2L1: 220uH, inductor-neosid:SD12-1000
- removed 2R2: 180R, resistor:R-EU_R0805
- removed C14: 100n, resistor:C-EUC0805K
- removed C16: 50u, resistor:CPOL-EUE2.5-6
- removed IC1: 4011D, 40xx:4011D
- removed IC2: MC34063AD, mc34063:MC34063AD
- added C1: 10m, rcl:C-EUC1210
- added C3, C4: 100n, resistor:C-EUC0805K
- added D1: (no value), diode:DIODE-SMB
- added D10, D11, D12, D13, D14, D15, D6, D8, D9: (no value), diode:DIODE-SOD80C
- added DA1: MC34063AD, mc34063:MC34063AD
- added DD1: 4011D, 40xx:4011D
- added L1: 100u, rcl:L-US6000-XXX-RC
- added R10, R11, R12, R7, R8, R9: (no value), rcl:R-EU_R0805
- 2C2: value 0.47n -> 59
- 2R1: value 1R -> 2r5
- 2R3: value 18K -> 11k
- 2R4: value 56K -> 18k
- C2: value 100n -> 10m; device resistor:C-EUC0805K -> rcl:C-EUC1210
Connections:
- removed net +5V: 1C10.+, 1R15.1, 2D1.C, 2R4.2, C14.1
- removed net N$11: 1R15.2, C2.1
- removed net N$21: 2D1.A, 2L1.2, IC2.SWC
- removed net N$22: 2R2.2, IC2.DC
- removed net N$24: 2L1.1, 2R1.2, 2R2.1, IC2.IS
- removed net V+: 2R1.1, C15.1, C16.+, IC2.VCC
- new net +12V: 2R1.1, C15.1, C2.1, DA1.VCC
- new net N$13: R11.1, R2.1, R8.1, S1.B.G
- new net N$14: R12.1, R3.1, R9.1, S1.B.R
- new net N$15: D12.C, R9.2
- new net N$16: D11.C, R8.2
- new net N$17: D10.C, R7.2
- new net N$18: D15.C, R12.2
- new net N$20: D14.C, R11.2
- new net N$23: D13.C, R10.2
- new net N$26: D13.A, D14.A, D15.A, VT1.C
- new net N$27: D10.A, D11.A, D12.A, VT2.C
- new net N$28: D6.A, D8.A, D9.A, VT3.C
- net +3V3: now also 2R4.2, C1.1, C3.1, C4.1, DD1P.VDD, L1.2
- net GND: now also C1.2, C2.2, C3.2, C4.2, D1.A, DA1.GND, DD1P.VSS; no longer C16.-, IC2.GND, IC2.SWE
- net N$19: now also D1.C, DA1.SWE, L1.1; no longer 2C2.1, IC2.TC
- net N$25: now also DA1.FB; no longer IC2.FB
- net N$3: now also 2R1.2, DA1.DC, DA1.IS, DA1.SWC; no longer R1.2, VT1.C
- net N$4: now also R1.1, R10.1, R7.1, S1.B.B; no longer R2.2, VT2.C
- net N$5: now also 2C2.1, DA1.TC; no longer R3.2, VT3.C
- net N$6: now also D9.C, R3.2; no longer R1.1, S1.B.B
- net N$7: now also D8.C, R2.2; no longer R2.1, S1.B.G
- net N$8: now also D6.C, R1.2; no longer R3.1, S1.B.R
Other:
- moved on the sheet: 2C2, 2R1, 2R3, 2R4, C15, C2, R1, R2, R3, R4, R5, R6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

Commit message: 3
Parts:
- added 2C1: 59, resistor:C-EUC0805K
- added JP1, JP2: (no value), pinhead:PINHD-1X2
Connections:
- new net N$21: JP2.1, S1.A.SW2
- new net N$22: JP2.2, S1.A.SW1
- net +12V: now also JP1.1
- net GND: now also 2C1.2, JP1.2
- net N$5: now also 2C1.1
Other:
- moved on the sheet: C1, C3, C4, D1, DD1P, L1
Changed lines of the file:
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@@
 <part name="C4" library="resistor" deviceset="C-EU" device="C0805K" value="100n"/>
 <part name="U$2" library="lib-user" deviceset="GND" device=""/>
+<part name="JP1" library="pinhead" deviceset="PINHD-1X2" device=""/>
+<part name="U$3" library="lib-user" deviceset="GND" device=""/>
+<part name="P+2" library="supply1" deviceset="+12V" device=""/>
+<part name="JP2" library="pinhead" deviceset="PINHD-1X2" device=""/>
+<part name="2C1" library="resistor" deviceset="C-EU" device="C0805K" value="59"/>
 </parts>
 <sheets>
@@
 <instance part="DD1" gate="C" x="83.82" y="134.62"/>
 <instance part="DD1" gate="D" x="104.14" y="132.08"/>
-<instance part="DD1" gate="P" x="142.24" y="33.02"/>
+<instance part="DD1" gate="P" x="149.86" y="33.02"/>
 <instance part="VT1" gate="G$1" x="218.44" y="114.3"/>
 <instance part="VT2" gate="G$1" x="236.22" y="121.92"/>
@@
 <instance part="D15" gate="G$1" x="226.06" y="101.6" rot="R270"/>
 <instance part="U$1" gate="G$1" x="81.28" y="25.4"/>
-<instance part="D1" gate="G$1" x="88.9" y="35.56" rot="R90"/>
-<instance part="+3V2" gate="G$1" x="124.46" y="50.8" smashed="yes">
-<attribute name="VALUE" x="127" y="53.34" size="1.778" layer="96" rot="R180"/>
-</instance>
-<instance part="L1" gate="G$1" x="99.06" y="43.18" rot="R90"/>
-<instance part="C1" gate="G$1" x="109.22" y="38.1"/>
+<instance part="D1" gate="G$1" x="96.52" y="35.56" rot="R90"/>
+<instance part="+3V2" gate="G$1" x="132.08" y="50.8" smashed="yes">
+<attribute name="VALUE" x="134.62" y="53.34" size="1.778" layer="96" rot="R180"/>
+</instance>
+<instance part="L1" gate="G$1" x="106.68" y="43.18" rot="R90"/>
+<instance part="C1" gate="G$1" x="116.84" y="38.1"/>
 <instance part="C2" gate="G$1" x="15.24" y="33.02"/>
-<instance part="C3" gate="G$1" x="116.84" y="38.1"/>
+<instance part="C3" gate="G$1" x="124.46" y="38.1"/>
 <instance part="P+1" gate="1" x="15.24" y="60.96" smashed="yes">
 <attribute name="VALUE" x="12.7" y="63.5" size="1.778" layer="96"/>
 </instance>
-<instance part="C4" gate="G$1" x="132.08" y="35.56"/>
-<instance part="U$2" gate="G$1" x="142.24" y="20.32"/>
+<instance part="C4" gate="G$1" x="139.7" y="35.56"/>
+<instance part="U$2" gate="G$1" x="149.86" y="20.32"/>
+<instance part="JP1" gate="G$1" x="45.72" y="88.9"/>
+<instance part="U$3" gate="G$1" x="30.48" y="86.36"/>
+<instance part="P+2" gate="1" x="30.48" y="96.52" smashed="yes">
+<attribute name="VALUE" x="27.94" y="99.06" size="1.778" layer="96"/>
+</instance>
+<instance part="JP2" gate="G$1" x="83.82" y="162.56"/>
+<instance part="2C1" gate="G$1" x="88.9" y="35.56" smashed="yes">
+<attribute name="NAME" x="87.884" y="48.641" size="1.778" layer="95"/>
+<attribute name="VALUE" x="87.884" y="46.101" size="1.778" layer="96"/>
+</instance>
 </instances>
 <busses>
@@
 <wire x1="81.28" y1="27.94" x2="88.9" y2="27.94" width="0.1524" layer="91"/>
 <pinref part="D1" gate="G$1" pin="A"/>
-<wire x1="88.9" y1="27.94" x2="88.9" y2="33.02" width="0.1524" layer="91"/>
+<wire x1="88.9" y1="27.94" x2="96.52" y2="27.94" width="0.1524" layer="91"/>
+<wire x1="96.52" y1="27.94" x2="96.52" y2="33.02" width="0.1524" layer="91"/>
 <junction x="81.28" y="27.94"/>
-<wire x1="88.9" y1="27.94" x2="109.22" y2="27.94" width="0.1524" layer="91"/>
+<wire x1="96.52" y1="27.94" x2="116.84" y2="27.94" width="0.1524" layer="91"/>
 <pinref part="C1" gate="G$1" pin="2"/>
-<wire x1="109.22" y1="27.94" x2="109.22" y2="33.02" width="0.1524" layer="91"/>
-<wire x1="109.22" y1="27.94" x2="116.84" y2="27.94" width="0.1524" layer="91"/>
+<wire x1="116.84" y1="27.94" x2="116.84" y2="33.02" width="0.1524" layer="91"/>
+<wire x1="116.84" y1="27.94" x2="124.46" y2="27.94" width="0.1524" layer="91"/>
 <pinref part="C3" gate="G$1" pin="2"/>
-<wire x1="116.84" y1="27.94" x2="116.84" y2="33.02" width="0.1524" layer="91"/>
-<junction x="109.22" y="27.94"/>
+<wire x1="124.46" y1="27.94" x2="124.46" y2="33.02" width="0.1524" layer="91"/>
+<junction x="116.84" y="27.94"/>
+<junction x="96.52" y="27.94"/>
+<pinref part="2C1" gate="G$1" pin="2"/>
+<wire x1="88.9" y1="30.48" x2="88.9" y2="27.94" width="0.1524" layer="91"/>
 <junction x="88.9" y="27.94"/>
 </segment>
 <segment>
 <pinref part="C4" gate="G$1" pin="2"/>
-<wire x1="132.08" y1="30.48" x2="132.08" y2="22.86" width="0.1524" layer="91"/>
-<wire x1="132.08" y1="22.86" x2="142.24" y2="22.86" width="0.1524" layer="91"/>
+<wire x1="139.7" y1="30.48" x2="139.7" y2="22.86" width="0.1524" layer="91"/>
+<wire x1="139.7" y1="22.86" x2="149.86" y2="22.86" width="0.1524" layer="91"/>
 <pinref part="DD1" gate="P" pin="VSS"/>
-<wire x1="142.24" y1="22.86" x2="142.24" y2="25.4" width="0.1524" layer="91"/>
+<wire x1="149.86" y1="22.86" x2="149.86" y2="25.4" width="0.1524" layer="91"/>
 <pinref part="U$2" gate="G$1" pin="GND"/>
-<wire x1="142.24" y1="22.86" x2="142.24" y2="20.32" width="0.1524" layer="91"/>
-<junction x="142.24" y="22.86"/>
+<wire x1="149.86" y1="22.86" x2="149.86" y2="20.32" width="0.1524" layer="91"/>
+<junction x="149.86" y="22.86"/>
+</segment>
+<segment>
+<pinref part="U$3" gate="G$1" pin="GND"/>
+<wire x1="30.48" y1="86.36" x2="30.48" y2="88.9" width="0.1524" layer="91"/>
+<pinref part="JP1" gate="G$1" pin="2"/>
+<wire x1="30.48" y1="88.9" x2="43.18" y2="88.9" width="0.1524" layer="91"/>
 </segment>
 </net>
@@
 <segment>
 <pinref part="2R4" gate="G$1" pin="2"/>
-<wire x1="58.42" y1="17.78" x2="124.46" y2="17.78" width="0.1524" layer="91"/>
+<wire x1="58.42" y1="17.78" x2="132.08" y2="17.78" width="0.1524" layer="91"/>
 <pinref part="+3V2" gate="G$1" pin="+3V3"/>
-<wire x1="124.46" y1="17.78" x2="124.46" y2="43.18" width="0.1524" layer="91"/>
+<wire x1="132.08" y1="17.78" x2="132.08" y2="43.18" width="0.1524" layer="91"/>
 <pinref part="L1" gate="G$1" pin="2"/>
-<wire x1="124.46" y1="43.18" x2="124.46" y2="48.26" width="0.1524" layer="91"/>
-<wire x1="106.68" y1="43.18" x2="109.22" y2="43.18" width="0.1524" layer="91"/>
+<wire x1="132.08" y1="43.18" x2="132.08" y2="48.26" width="0.1524" layer="91"/>
+<wire x1="114.3" y1="43.18" x2="116.84" y2="43.18" width="0.1524" layer="91"/>
+<junction x="132.08" y="43.18"/>
+<pinref part="C1" gate="G$1" pin="1"/>
+<wire x1="116.84" y1="43.18" x2="124.46" y2="43.18" width="0.1524" layer="91"/>
+<wire x1="124.46" y1="43.18" x2="132.08" y2="43.18" width="0.1524" layer="91"/>
+<wire x1="116.84" y1="40.64" x2="116.84" y2="43.18" width="0.1524" layer="91"/>
+<pinref part="C3" gate="G$1" pin="1"/>
+<wire x1="124.46" y1="40.64" x2="124.46" y2="43.18" width="0.1524" layer="91"/>
+<junction x="116.84" y="43.18"/>
 <junction x="124.46" y="43.18"/>
-<pinref part="C1" gate="G$1" pin="1"/>
-<wire x1="109.22" y1="43.18" x2="116.84" y2="43.18" width="0.1524" layer="91"/>
-<wire x1="116.84" y1="43.18" x2="124.46" y2="43.18" width="0.1524" layer="91"/>
-<wire x1="109.22" y1="40.64" x2="109.22" y2="43.18" width="0.1524" layer="91"/>
-<pinref part="C3" gate="G$1" pin="1"/>
-<wire x1="116.84" y1="40.64" x2="116.84" y2="43.18" width="0.1524" layer="91"/>
-<junction x="109.22" y="43.18"/>
-<junction x="116.84" y="43.18"/>
-<wire x1="124.46" y1="43.18" x2="132.08" y2="43.18" width="0.1524" layer="91"/>
+<wire x1="132.08" y1="43.18" x2="139.7" y2="43.18" width="0.1524" layer="91"/>
 <pinref part="C4" gate="G$1" pin="1"/>
-<wire x1="132.08" y1="43.18" x2="132.08" y2="38.1" width="0.1524" layer="91"/>
+<wire x1="139.7" y1="43.18" x2="139.7" y2="38.1" width="0.1524" layer="91"/>
 <pinref part="DD1" gate="P" pin="VDD"/>
-<wire x1="142.24" y1="40.64" x2="142.24" y2="43.18" width="0.1524" layer="91"/>
-<wire x1="142.24" y1="43.18" x2="132.08" y2="43.18" width="0.1524" layer="91"/>
-<junction x="132.08" y="43.18"/>
+<wire x1="149.86" y1="40.64" x2="149.86" y2="43.18" width="0.1524" layer="91"/>
+<wire x1="149.86" y1="43.18" x2="139.7" y2="43.18" width="0.1524" layer="91"/>
+<junction x="139.7" y="43.18"/>
 </segment>
 </net>
@@
 <wire x1="68.58" y1="40.64" x2="81.28" y2="40.64" width="0.1524" layer="91"/>
 <wire x1="81.28" y1="40.64" x2="81.28" y2="38.1" width="0.1524" layer="91"/>
+<pinref part="2C1" gate="G$1" pin="1"/>
+<wire x1="88.9" y1="38.1" x2="88.9" y2="40.64" width="0.1524" layer="91"/>
+<wire x1="88.9" y1="40.64" x2="81.28" y2="40.64" width="0.1524" layer="91"/>
+<junction x="81.28" y="40.64"/>
 </segment>
 </net>
@@
 <segment>
 <pinref part="DA1" gate="G$1" pin="SWE"/>
-<wire x1="68.58" y1="43.18" x2="88.9" y2="43.18" width="0.1524" layer="91"/>
+<wire x1="68.58" y1="43.18" x2="96.52" y2="43.18" width="0.1524" layer="91"/>
 <pinref part="D1" gate="G$1" pin="C"/>
-<wire x1="88.9" y1="43.18" x2="88.9" y2="38.1" width="0.1524" layer="91"/>
+<wire x1="96.52" y1="43.18" x2="96.52" y2="38.1" width="0.1524" layer="91"/>
 <pinref part="L1" gate="G$1" pin="1"/>
-<wire x1="88.9" y1="43.18" x2="91.44" y2="43.18" width="0.1524" layer="91"/>
-<junction x="88.9" y="43.18"/>
+<wire x1="96.52" y1="43.18" x2="99.06" y2="43.18" width="0.1524" layer="91"/>
+<junction x="96.52" y="43.18"/>
 </segment>
 </net>
@@
 <junction x="15.24" y="53.34"/>
 </segment>
-</net>
+<segment>
+<pinref part="JP1" gate="G$1" pin="1"/>
+<wire x1="43.18" y1="91.44" x2="30.48" y2="91.44" width="0.1524" layer="91"/>
+<pinref part="P+2" gate="1" pin="+12V"/>
+<wire x1="30.48" y1="91.44" x2="30.48" y2="93.98" width="0.1524" layer="91"/>
+</segment>
+</net>
+<net name="N$21" class="0">
+<segment>
+<pinref part="JP2" gate="G$1" pin="1"/>
+<pinref part="S1" gate=".A" pin="SW2"/>
+<wire x1="81.28" y1="165.1" x2="73.66" y2="165.1" width="0.1524" layer="91"/>
+</segment>
+</net>
+<net name="N$22" class="0">
+<segment>
+<pinref part="JP2" gate="G$1" pin="2"/>
+<wire x1="81.28" y1="162.56" x2="60.96" y2="162.56" width="0.1524" layer="91"/>
+<wire x1="60.96" y1="162.56" x2="60.96" y2="165.1" width="0.1524" layer="91"/>
+<pinref part="S1" gate=".A" pin="SW1"/>
+<wire x1="60.96" y1="165.1" x2="63.5" y2="165.1" width="0.1524" layer="91"/>
+</segment>
+</net>

Commit message: 4
Connections:
- removed net N$17: D10.C, R7.2
- new net N$11: D10.A, R7.1
- net N$13: now also D11.C; no longer R8.1
- net N$16: now also D11.A, R8.1; no longer D11.C, R8.2
- net N$27: now also R7.2, R8.2; no longer D10.A, D11.A
- net N$4: now also D10.C; no longer R7.1
Other:
- note added: "POWER"
- note added: "SSD"
- note added: "STAND"
- moved on the sheet: D10, D11, DD1D, R7, R8
Changed lines of the file:
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@@
 <sheet>
 <plain>
+<text x="261.62" y="129.54" size="1.778" layer="91">SSD</text>
+<text x="241.3" y="121.92" size="1.778" layer="91">POWER</text>
+<text x="223.52" y="114.3" size="1.778" layer="91">STAND</text>
 </plain>
 <instances>
@@
 <instance part="DD1" gate="B" x="58.42" y="134.62"/>
 <instance part="DD1" gate="C" x="83.82" y="134.62"/>
-<instance part="DD1" gate="D" x="104.14" y="132.08"/>
+<instance part="DD1" gate="D" x="180.34" y="114.3"/>
 <instance part="DD1" gate="P" x="149.86" y="33.02"/>
 <instance part="VT1" gate="G$1" x="218.44" y="114.3"/>
@@
 <instance part="D8" gate="G$1" x="256.54" y="101.6" rot="R270"/>
 <instance part="D9" gate="G$1" x="261.62" y="101.6" rot="R270"/>
-<instance part="R7" gate="G$1" x="233.68" y="91.44" rot="R90"/>
-<instance part="R8" gate="G$1" x="238.76" y="91.44" rot="R90"/>
+<instance part="R7" gate="G$1" x="233.68" y="99.06" rot="R90"/>
+<instance part="R8" gate="G$1" x="238.76" y="99.06" rot="R90"/>
 <instance part="R9" gate="G$1" x="243.84" y="91.44" rot="R90"/>
-<instance part="D10" gate="G$1" x="233.68" y="101.6" rot="R270"/>
-<instance part="D11" gate="G$1" x="238.76" y="101.6" rot="R270"/>
+<instance part="D10" gate="G$1" x="233.68" y="88.9" rot="R270"/>
+<instance part="D11" gate="G$1" x="238.76" y="88.9" rot="R270"/>
 <instance part="D12" gate="G$1" x="243.84" y="101.6" rot="R270"/>
 <instance part="R10" gate="G$1" x="215.9" y="91.44" rot="R90"/>
@@
 <wire x1="251.46" y1="73.66" x2="251.46" y2="86.36" width="0.1524" layer="91"/>
 <wire x1="251.46" y1="73.66" x2="233.68" y2="73.66" width="0.1524" layer="91"/>
-<pinref part="R7" gate="G$1" pin="1"/>
-<wire x1="233.68" y1="73.66" x2="233.68" y2="86.36" width="0.1524" layer="91"/>
 <junction x="233.68" y="73.66"/>
 <wire x1="233.68" y1="73.66" x2="215.9" y2="73.66" width="0.1524" layer="91"/>
@@
 <pinref part="S1" gate=".B" pin="B"/>
 <wire x1="233.68" y1="71.12" x2="233.68" y2="73.66" width="0.1524" layer="91"/>
+<pinref part="D10" gate="G$1" pin="C"/>
+<wire x1="233.68" y1="86.36" x2="233.68" y2="73.66" width="0.1524" layer="91"/>
 </segment>
 </net>
@@
 <wire x1="238.76" y1="78.74" x2="220.98" y2="78.74" width="0.1524" layer="91"/>
 <wire x1="256.54" y1="78.74" x2="256.54" y2="86.36" width="0.1524" layer="91"/>
-<pinref part="R8" gate="G$1" pin="1"/>
-<wire x1="238.76" y1="78.74" x2="238.76" y2="86.36" width="0.1524" layer="91"/>
 <junction x="238.76" y="78.74"/>
 <pinref part="R11" gate="G$1" pin="1"/>
@@
 <pinref part="S1" gate=".B" pin="G"/>
 <wire x1="238.76" y1="71.12" x2="238.76" y2="78.74" width="0.1524" layer="91"/>
+<pinref part="D11" gate="G$1" pin="C"/>
+<wire x1="238.76" y1="86.36" x2="238.76" y2="78.74" width="0.1524" layer="91"/>
 </segment>
 </net>
@@
 </segment>
 </net>
-<net name="N$16" class="0">
-<segment>
-<pinref part="D11" gate="G$1" pin="C"/>
-<pinref part="R8" gate="G$1" pin="2"/>
-<wire x1="238.76" y1="99.06" x2="238.76" y2="96.52" width="0.1524" layer="91"/>
-</segment>
-</net>
-<net name="N$17" class="0">
-<segment>
-<pinref part="D10" gate="G$1" pin="C"/>
-<pinref part="R7" gate="G$1" pin="2"/>
-<wire x1="233.68" y1="99.06" x2="233.68" y2="96.52" width="0.1524" layer="91"/>
-</segment>
-</net>
 <net name="N$18" class="0">
 <segment>
@@
 <net name="N$27" class="0">
 <segment>
-<pinref part="D10" gate="G$1" pin="A"/>
-<wire x1="233.68" y1="104.14" x2="233.68" y2="106.68" width="0.1524" layer="91"/>
 <wire x1="233.68" y1="106.68" x2="238.76" y2="106.68" width="0.1524" layer="91"/>
-<pinref part="D11" gate="G$1" pin="A"/>
-<wire x1="238.76" y1="106.68" x2="238.76" y2="104.14" width="0.1524" layer="91"/>
 <wire x1="238.76" y1="106.68" x2="243.84" y2="106.68" width="0.1524" layer="91"/>
 <pinref part="D12" gate="G$1" pin="A"/>
@@
 <pinref part="VT2" gate="G$1" pin="C"/>
 <wire x1="238.76" y1="116.84" x2="238.76" y2="106.68" width="0.1524" layer="91"/>
+<pinref part="R7" gate="G$1" pin="2"/>
+<wire x1="233.68" y1="104.14" x2="233.68" y2="106.68" width="0.1524" layer="91"/>
+<pinref part="R8" gate="G$1" pin="2"/>
+<wire x1="238.76" y1="104.14" x2="238.76" y2="106.68" width="0.1524" layer="91"/>
 </segment>
 </net>
@@
 </segment>
 </net>
+<net name="N$11" class="0">
+<segment>
+<pinref part="D10" gate="G$1" pin="A"/>
+<pinref part="R7" gate="G$1" pin="1"/>
+<wire x1="233.68" y1="91.44" x2="233.68" y2="93.98" width="0.1524" layer="91"/>
+</segment>
+</net>
+<net name="N$16" class="0">
+<segment>
+<pinref part="R8" gate="G$1" pin="1"/>
+<pinref part="D11" gate="G$1" pin="A"/>
+<wire x1="238.76" y1="93.98" x2="238.76" y2="91.44" width="0.1524" layer="91"/>
+</segment>
+</net>

Commit message: 6
Connections:
- removed net N$23: D13.C, R10.2
- new net N$17: D15.A, R12.1
- net N$13: now also D14.C, D8.C; no longer R11.1, R2.1
- net N$14: now also D12.C, D15.C, D9.C; no longer R12.1, R3.1, R9.1
- net N$15: now also D12.A, R9.1; no longer D12.C, R9.2
- net N$18: now also D14.A, R11.1; no longer D15.C, R12.2
- net N$20: now also D13.A, R10.1; no longer D14.C, R11.2
- net N$26: now also R10.2, R11.2, R12.2; no longer D13.A, D14.A, D15.A
- net N$27: now also R9.2; no longer D12.A
- net N$28: now also R1.2, R2.2, R3.2; no longer D6.A, D8.A, D9.A
- net N$4: now also D13.C, D6.C; no longer R1.1, R10.1
- net N$6: now also D9.A, R3.1; no longer D9.C, R3.2
- net N$7: now also D8.A, R2.1; no longer D8.C, R2.2
- net N$8: now also D6.A, R1.1; no longer D6.C, R1.2
Other:
- moved on the sheet: D12, D13, D14, D15, D6, D8, D9, R1, R10, R11, R12, R2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

Commit message: 7
Parts:
- added 2R2: 2r5, resistor:R-EU_R0805
- added R13: 10, rcl:R-EU_R0805
- added R14: (no value), rcl:R-EU_R1206W
- R4, R6: device rcl:R-EU_R0805 -> rcl:R-EU_R1206W
- VT1, VT2, VT3: device m_transistor:BJT_PNP_TO126_V_ECB -> m_transistor:BJT_PNP_TO-92_EBC
Connections:
- new net N$23: R13.2, S1.B.RGB-
- new net N$24: D10.C, R14.2
- new net OUT1: DD1C.O, R4.1
- new net OUT2: DD1C.I0, DD1D.O, R5.1
- new net OUT3: DD1B.O, DD1C.I1, DD1D.I1, R6.1
- new net POWER: DD1D.I0
- new net SSD: DD1B.I0, DD1B.I1
- net +12V: now also 2R2.1
- net GND: now also R13.1; no longer S1.B.RGB-
- net N$3: now also 2R2.2
- net N$4: now also R14.1; no longer D10.C
Other:
- moved on the sheet: D10, D11, D12, D13, D14, D15, D6, D8, D9, DD1A, DD1B, DD1C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

Commit message: 8
Parts:
- removed 2R3: 11k, resistor:R-EU_R0805
- removed 2R4: 18k, resistor:R-EU_R0805
- removed C15: 100n, resistor:C-EUC0805K
- removed D10: (no value), diode:DIODE-SOD80C
- removed R14: (no value), rcl:R-EU_R1206W
- removed R5, R7: (no value), rcl:R-EU_R0805
- added 1RG, 1RR, 2RB: (no value), rcl:R-EU_R0805
- added 2VDB: (no value), diode:DIODE-SOD80C
- added C5: 10m, rcl:C-EUC1210
- added J1: (no value), rcl:R-EU_R1206W
- added R1A: 2r5, resistor:R-EU_R0805
- 2R1: value 2r5 -> (none); device resistor:R-EU_R0805 -> rcl:R-EU_R0805
- C2: value 10m -> 100n; device rcl:C-EUC1210 -> resistor:C-EUC0805K
- R2: value (none) -> 11k; device rcl:R-EU_R0805 -> resistor:R-EU_R0805
- R3: value (none) -> 18k; device rcl:R-EU_R0805 -> resistor:R-EU_R0805
- renumbered 2C1 to C3B, 2C2 to C3A, 2R2 to R1B, C3 to C6, C4 to C7, D1 to VD1, D11 to 2VDG, D12 to 2VDR, D13 to 3VDB, D14 to 3VDG, D15 to 3VDR, D6 to 1VDB, D8 to 1VDG, D9 to 1VDR, R1 to 1RB, R10 to 3RB, R11 to 3RG, R12 to 3RR, R4 to 1R1, R6 to 3R1, R8 to 2RG, R9 to 2RR
Connections:
- net OUT1 renamed OUT_SLED
- net OUT3 renamed OUT_DSLED
- net POWER renamed PWRLED
- net SSD renamed DSKLED
- removed net OUT2: DD1C.I0, DD1D.O, R5.1
- new net OUT_PWLED: 2R1.1, DD1C.I0, DD1D.O
- net +12V: now also C1.1, R1A.1; no longer 2R1.1, C15.1
- net +3V3: now also C5.1, R3.2; no longer 2R4.2, C1.1
- net GND: now also C5.2, R2.1; no longer 2R3.1, C15.2
- net N$10: now also 2R1.2; no longer R5.2
- net N$11: now also 2RB.1, 2VDB.A; no longer D10.A, R7.1
- net N$24: now also 2VDB.C, J1.2; no longer D10.C, R14.2
- net N$25: now also R2.2, R3.1; no longer 2R3.2, 2R4.1
- net N$27: now also 2RB.2; no longer R7.2
- net N$28: now also 1RG.2, 1RR.2; no longer R2.2, R3.2
- net N$3: now also R1A.2; no longer 2R1.2
- net N$4: now also J1.1; no longer R14.1
- net N$6: now also 1RR.1; no longer R3.1
- net N$7: now also 1RG.1; no longer R2.1
Other:
- moved on the sheet: 2R1, C1, C2, DD1A, R2, R3

Commit message: 11
Parts:
- added +12V: CON_2P, DSS:CON_2P
- added JP5, JP6: (no value), pinhead:PINHD-1X1
- 2R1: device rcl:R-EU_R0805 -> rcl:R-EU_R1206W
- JP1: device pinhead:PINHD-1X2 -> pinhead:PINHD-1X1
- R1B: value 2r5 -> (none)
Connections:
- net +12V: now also +12V.1; no longer JP1.1
- net +3V3: now also DD1A.I0, DD1A.I1
- net DSKLED: now also DD1C.I0, DD1C.I1, JP6.1; no longer DD1B.I0, DD1B.I1
- net GND: now also +12V.2; no longer JP1.2
- net OUT_DSLED: now also DD1B.I0, DD1C.O; no longer DD1B.O, DD1C.I1
- net OUT_PWLED: now also DD1B.I1; no longer DD1C.I0
- net OUT_SLED: now also DD1B.O; no longer DD1C.O
- net PWRLED: now also JP5.1
Other:
- moved on the sheet: C1, C2, C3A, C3B, C5, C6, C7, DA1, DD1A, DD1B, DD1C, DD1P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

Commit message: 12
Parts:
- VT1, VT2, VT3: value KT561 -> KT3107
- renumbered R13 to RC1
Other:
- moved on the sheet: DD1A, DD1B, DD1C, DD1D, JP1, JP2, JP5, JP6, S1
