File: pc2_key.sch (EAGLE design)
At the start: 47 parts

Commit message: 14
Parts:
- removed JP1, JP5, JP6: (no value), pinhead:PINHD-1X1
- added HDDLED, PWRLED: (no value), pinhead:PINHD-1X1
- added R1: (no value), rcl:R-EU_M0805
- added R4: (no value), rcl:R-EU_R1206W
- R1A, R1B: device resistor:R-EU_R0805 -> resistor:R-EU_R1206
Connections:
- net DSKLED: now also HDDLED.1, R4.2; no longer JP6.1
- net GND: now also R1.1, R4.1
- net PWRLED: now also PWRLED.1, R1.2; no longer JP5.1
Changed lines of the file:
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@@
 <part name="DA1" library="mc34063" deviceset="MC34063" device="AD"/>
 <part name="C3A" library="resistor" deviceset="C-EU" device="C0805K" value="59"/>
-<part name="R1A" library="resistor" deviceset="R-EU_" device="R0805" value="2r5"/>
+<part name="R1A" library="resistor" deviceset="R-EU_" device="R1206" value="2r5"/>
 <part name="U$13" library="lib-user" deviceset="GND" device=""/>
 <part name="R2" library="resistor" deviceset="R-EU_" device="R0805" value="11k"/>
@@
 <part name="RC1" library="rcl" deviceset="R-EU_" device="R0805" value="10"/>
 <part name="J1" library="rcl" deviceset="R-EU_" device="R1206W"/>
-<part name="R1B" library="resistor" deviceset="R-EU_" device="R0805"/>
-<part name="JP5" library="pinhead" deviceset="PINHD-1X1" device=""/>
-<part name="JP6" library="pinhead" deviceset="PINHD-1X1" device=""/>
+<part name="R1B" library="resistor" deviceset="R-EU_" device="R1206"/>
+<part name="PWRLED" library="pinhead" deviceset="PINHD-1X1" device=""/>
+<part name="HDDLED" library="pinhead" deviceset="PINHD-1X1" device=""/>
 <part name="+12V" library="DSS" deviceset="CON_2P" device="" value=""/>
-<part name="JP1" library="pinhead" deviceset="PINHD-1X1" device=""/>
 <part name="+3V3" library="supply1" deviceset="+3V3" device=""/>
+<part name="R1" library="rcl" deviceset="R-EU_" device="M0805"/>
+<part name="R4" library="rcl" deviceset="R-EU_" device="R1206W"/>
+<part name="U$3" library="lib-user" deviceset="GND" device=""/>
+<part name="U$4" library="lib-user" deviceset="GND" device=""/>
 </parts>
 <sheets>
@@
 <instance part="J1" gate="G$1" x="231.14" y="109.22" rot="R90"/>
 <instance part="R1B" gate="G$1" x="35.56" y="48.26"/>
-<instance part="JP5" gate="G$1" x="129.54" y="114.3" rot="MR0"/>
-<instance part="JP6" gate="G$1" x="129.54" y="91.44" rot="MR0"/>
+<instance part="PWRLED" gate="G$1" x="124.46" y="114.3" rot="MR0"/>
+<instance part="HDDLED" gate="G$1" x="124.46" y="91.44" rot="MR0"/>
 <instance part="+12V" gate="G$1" x="10.16" y="30.48" smashed="yes" rot="MR180">
 <attribute name="VALUE" x="7.62" y="38.1" size="1.778" layer="96" rot="MR180"/>
 <attribute name="NAME" x="15.24" y="36.322" size="1.778" layer="95" rot="MR0"/>
 </instance>
-<instance part="JP1" gate="G$1" x="129.54" y="104.14" rot="MR0"/>
 <instance part="+3V3" gate="G$1" x="152.4" y="139.7" smashed="yes">
 <attribute name="VALUE" x="154.94" y="142.24" size="1.778" layer="96" rot="R180"/>
 </instance>
+<instance part="R1" gate="G$1" x="134.62" y="106.68" rot="R90"/>
+<instance part="R4" gate="G$1" x="134.62" y="83.82" rot="R90"/>
+<instance part="U$3" gate="G$1" x="134.62" y="76.2"/>
+<instance part="U$4" gate="G$1" x="134.62" y="99.06"/>
 </instances>
 <busses>
@@
 <wire x1="236.22" y1="68.58" x2="236.22" y2="66.04" width="0.1524" layer="91"/>
 </segment>
+<segment>
+<pinref part="R1" gate="G$1" pin="1"/>
+<pinref part="U$4" gate="G$1" pin="GND"/>
+<wire x1="134.62" y1="101.6" x2="134.62" y2="99.06" width="0.1524" layer="91"/>
+</segment>
+<segment>
+<pinref part="R4" gate="G$1" pin="1"/>
+<pinref part="U$3" gate="G$1" pin="GND"/>
+<wire x1="134.62" y1="78.74" x2="134.62" y2="76.2" width="0.1524" layer="91"/>
+</segment>
 </net>
 <net name="N$25" class="0">
@@
 <pinref part="DD1" gate="C" pin="I1"/>
 <pinref part="DD1" gate="C" pin="I0"/>
-<label x="139.7" y="91.44" size="1.778" layer="95"/>
+<label x="139.7" y="93.98" size="1.778" layer="95"/>
 <junction x="152.4" y="91.44"/>
 <wire x1="154.94" y1="88.9" x2="152.4" y2="88.9" width="0.1524" layer="91"/>
@@
 <wire x1="152.4" y1="91.44" x2="152.4" y2="93.98" width="0.1524" layer="91"/>
 <wire x1="152.4" y1="93.98" x2="154.94" y2="93.98" width="0.1524" layer="91"/>
-<pinref part="JP6" gate="G$1" pin="1"/>
-<wire x1="132.08" y1="91.44" x2="137.16" y2="91.44" width="0.1524" layer="91"/>
-<junction x="137.16" y="91.44"/>
-<wire x1="137.16" y1="91.44" x2="152.4" y2="91.44" width="0.1524" layer="91"/>
+<pinref part="HDDLED" gate="G$1" pin="1"/>
+<wire x1="127" y1="91.44" x2="132.08" y2="91.44" width="0.1524" layer="91"/>
+<junction x="132.08" y="91.44"/>
+<wire x1="132.08" y1="91.44" x2="134.62" y2="91.44" width="0.1524" layer="91"/>
+<pinref part="R4" gate="G$1" pin="2"/>
+<wire x1="134.62" y1="91.44" x2="152.4" y2="91.44" width="0.1524" layer="91"/>
+<wire x1="134.62" y1="88.9" x2="134.62" y2="91.44" width="0.1524" layer="91"/>
+<junction x="134.62" y="91.44"/>
 </segment>
 </net>
@@
 <segment>
 <pinref part="DD1" gate="D" pin="I0"/>
-<wire x1="154.94" y1="114.3" x2="137.16" y2="114.3" width="0.1524" layer="91"/>
+<wire x1="154.94" y1="114.3" x2="134.62" y2="114.3" width="0.1524" layer="91"/>
 <label x="139.7" y="114.3" size="1.778" layer="95"/>
-<pinref part="JP5" gate="G$1" pin="1"/>
-<wire x1="132.08" y1="114.3" x2="137.16" y2="114.3" width="0.1524" layer="91"/>
-<junction x="137.16" y="114.3"/>
-</segment>
-</net>
+<pinref part="PWRLED" gate="G$1" pin="1"/>
+<wire x1="134.62" y1="114.3" x2="132.08" y2="114.3" width="0.1524" layer="91"/>
+<wire x1="127" y1="114.3" x2="132.08" y2="114.3" width="0.1524" layer="91"/>
+<junction x="132.08" y="114.3"/>
+<pinref part="R1" gate="G$1" pin="2"/>
+<wire x1="134.62" y1="111.76" x2="134.62" y2="114.3" width="0.1524" layer="91"/>
+<junction x="134.62" y="114.3"/>
+</segment>
+</net>

Commit message: 15
Parts:
- added C3: 10m, rcl:C-EUC1210
- added L2: (no value), rcl:L-USL1812
Connections:
- net +12V renamed N$30
- new net N$29: C5.1, C6.1, L1.2, L2.1, R3.2
- net +3V3: now also C3.1, L2.2; no longer C5.1, C6.1, L1.2, R3.2
- net GND: now also C3.2
Other:
- moved on the sheet: +12V, 1R1, 1RB, 1RG, 1RR, 1VDB, 1VDG, 1VDR, 2R1, 2RB, 2RG, 2RR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

Commit message: 17
Parts:
- added GND: (no value), pinhead:PINHD-1X1
Connections:
- net GND: now also GND.1
Changed lines of the file:
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@@
 <part name="L2" library="rcl" deviceset="L-US" device="L1812"/>
 <part name="C3" library="rcl" deviceset="C-EU" device="C1210" value="10m"/>
+<part name="GND" library="pinhead" deviceset="PINHD-1X1" device=""/>
 </parts>
 <sheets>
@@
 <instance part="R1" gate="G$1" x="33.02" y="157.48" rot="R90"/>
 <instance part="R4" gate="G$1" x="33.02" y="134.62" rot="R90"/>
-<instance part="U$3" gate="G$1" x="33.02" y="127"/>
+<instance part="U$3" gate="G$1" x="33.02" y="124.46"/>
 <instance part="U$4" gate="G$1" x="33.02" y="149.86"/>
 <instance part="L2" gate="G$1" x="114.3" y="35.56" rot="R90"/>
 <instance part="C3" gate="G$1" x="124.46" y="27.94"/>
+<instance part="GND" gate="G$1" x="22.86" y="127" rot="MR0"/>
 </instances>
 <busses>
@@
 <pinref part="U$3" gate="G$1" pin="GND"/>
 <wire x1="33.02" y1="129.54" x2="33.02" y2="127" width="0.1524" layer="91"/>
+<pinref part="GND" gate="G$1" pin="1"/>
+<wire x1="33.02" y1="127" x2="33.02" y2="124.46" width="0.1524" layer="91"/>
+<wire x1="25.4" y1="127" x2="33.02" y2="127" width="0.1524" layer="91"/>
+<junction x="33.02" y="127"/>
 </segment>
 </net>

Commit message: 18
Parts:
- L1: device rcl:L-US6000-XXX-RC -> inductor-neosid:SD12K100
- renumbered JP2 to SW1
Changed lines of the file:
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@@
 <part name="VD1" library="diode" deviceset="DIODE-" device="SMB"/>
 <part name="+3V2" library="supply1" deviceset="+3V3" device=""/>
-<part name="L1" library="rcl" deviceset="L-US" device="6000-XXX-RC" value="100u"/>
+<part name="L1" library="inductor-neosid" deviceset="SD12" device="K100" value="100u"/>
 <part name="C5" library="rcl" deviceset="C-EU" device="C1210" value="10m"/>
 <part name="C1" library="rcl" deviceset="C-EU" device="C1210" value="10m"/>
@@
 <part name="C7" library="resistor" deviceset="C-EU" device="C0805K" value="100n"/>
 <part name="U$2" library="lib-user" deviceset="GND" device=""/>
-<part name="JP2" library="pinhead" deviceset="PINHD-1X2" device=""/>
+<part name="SW1" library="pinhead" deviceset="PINHD-1X2" device=""/>
 <part name="C3B" library="resistor" deviceset="C-EU" device="C0805K" value="59"/>
 <part name="RC1" library="rcl" deviceset="R-EU_" device="R0805" value="10"/>
@@
 <attribute name="VALUE" x="134.62" y="43.18" size="1.778" layer="96" rot="R180"/>
 </instance>
-<instance part="L1" gate="G$1" x="116.84" y="71.12" smashed="yes" rot="R90">
+<instance part="L1" gate="G$1" x="116.84" y="71.12" smashed="yes">
 <attribute name="NAME" x="114.3" y="74.93" size="1.778" layer="95" rot="R180"/>
 <attribute name="VALUE" x="121.92" y="74.93" size="1.778" layer="96" rot="R180"/>
@@
 <instance part="C7" gate="G$1" x="132.08" y="27.94"/>
 <instance part="U$2" gate="G$1" x="142.24" y="12.7"/>
-<instance part="JP2" gate="G$1" x="68.58" y="116.84"/>
+<instance part="SW1" gate="G$1" x="68.58" y="116.84"/>
 <instance part="C3B" gate="G$1" x="99.06" y="63.5" smashed="yes">
 <attribute name="NAME" x="98.044" y="76.581" size="1.778" layer="95"/>
@@
 <wire x1="106.68" y1="71.12" x2="106.68" y2="66.04" width="0.1524" layer="91"/>
 <pinref part="L1" gate="G$1" pin="1"/>
-<wire x1="106.68" y1="71.12" x2="109.22" y2="71.12" width="0.1524" layer="91"/>
+<wire x1="106.68" y1="71.12" x2="111.76" y2="71.12" width="0.1524" layer="91"/>
 <junction x="106.68" y="71.12"/>
 </segment>
@@
 <net name="N$21" class="0">
 <segment>
-<pinref part="JP2" gate="G$1" pin="1"/>
+<pinref part="SW1" gate="G$1" pin="1"/>
 <pinref part="S1" gate=".A" pin="SW2"/>
 <wire x1="66.04" y1="119.38" x2="58.42" y2="119.38" width="0.1524" layer="91"/>
@@
 <net name="N$22" class="0">
 <segment>
-<pinref part="JP2" gate="G$1" pin="2"/>
+<pinref part="SW1" gate="G$1" pin="2"/>
 <wire x1="66.04" y1="116.84" x2="45.72" y2="116.84" width="0.1524" layer="91"/>
 <wire x1="45.72" y1="116.84" x2="45.72" y2="119.38" width="0.1524" layer="91"/>
@@
 <junction x="134.62" y="71.12"/>
 <pinref part="L1" gate="G$1" pin="2"/>
-<wire x1="124.46" y1="71.12" x2="127" y2="71.12" width="0.1524" layer="91"/>
+<wire x1="121.92" y1="71.12" x2="127" y2="71.12" width="0.1524" layer="91"/>
 <wire x1="127" y1="71.12" x2="134.62" y2="71.12" width="0.1524" layer="91"/>
 <junction x="127" y="71.12"/>

Commit message: 18
Parts:
- added 3VDB1: LL4148, diode:DIODE-SOD80C
- added F1: (no value), fuse:SH32
- added J2: (no value), rcl:R-EU_R1206W
- added SJ1: (no value), jumper:SJ
- C3, C5: value 10m -> 22m
- L1: device inductor-neosid:SD12K100 -> ct-pack:L_LH7X10MM
- L2: value (none) -> 10mkhn; device rcl:L-USL1812 -> rcl:L-USPIS2816
Connections:
- new net N$32: 3VDB1.C, DD1A.O
- new net N$33: +12V.1, F1.1A
- new net N$34: DD1A.I0, DD1A.I1, J1.2
- net +3V3: no longer DD1A.I0, DD1A.I1
- net GND: now also SJ1.1
- net N$19: now also L1.2; no longer L1.1
- net N$21: now also 3VDB1.A, SJ1.2
- net N$24: now also J2.2; no longer J1.2
- net N$29: now also L1.1; no longer L1.2
- net N$30: now also F1.2A; no longer +12V.1
- net N$4: now also J2.1; no longer J1.1
- net PWRLED: now also J1.1
Other:
- moved on the sheet: +12V, C1, C2, C3, C3A, C3B, C5, C6, C7, DA1, DD1A, DD1B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

Commit message: 19
Parts:
- removed R1: (no value), rcl:R-EU_M0805
- added R5: 10k, rcl:R-EU_R1206W
- C3A: value 59 -> 68
- C3B: value 59 -> (none)
- J1, J2: value (none) -> 0
- R1A: value 2r5 -> 4R7
- R1B: value (none) -> 4R7
- R2: value 11k -> 8k2
- R3: value 18k -> 15k
- R4: value (none) -> 10k; device rcl:R-EU_R1206W -> rcl:R-EU_M0805
- renumbered C3 to C8
Connections:
- net +3V3 renamed VCC
- net N$25 renamed 1,25V
- net N$29 renamed 3V5
- net DSKLED: now also R5.2; no longer R4.2
- net GND: now also R5.1; no longer R1.1
- net PWRLED: now also R4.2; no longer R1.2
Other:
- note added: "3V5"
- moved on the sheet: R4

Commit message: 20
Parts:
- removed 3VDB1: LL4148, diode:DIODE-SOD80C
- removed HDDLED: (no value), pinhead:PINHD-1X1
- removed J1: 0, rcl:R-EU_R1206W
- removed SJ1: (no value), jumper:SJ
- added !HDDLED: (no value), pinhead:PINHD-1X1
- C1: value 10m -> 33m
- RC1: value 10 -> 22
Connections:
- net OUT_PWLED renamed !OUT_PWLED
- net OUT_SLED renamed !OUT_SLED
- removed net DSKLED: DD1C.I0, DD1C.I1, HDDLED.1, R5.2
- removed net N$32: 3VDB1.C, DD1A.O
- removed net N$34: DD1A.I0, DD1A.I1, J1.2
- removed net OUT_DSLED: 3R1.1, DD1B.I0, DD1C.O, DD1D.I1
- new net !DSKLED: !HDDLED.1, DD1C.I0, DD1C.I1, R5.2
- new net !OUT_DSLED: 3R1.1, DD1A.O, DD1B.I0, DD1D.I1
- new net N$29: DD1A.I0, DD1A.I1, DD1C.O
- net GND: no longer SJ1.1
- net N$21: no longer 3VDB1.A, SJ1.2
- net PWRLED: no longer J1.1
Other:
- moved on the sheet: DD1A, DD1B, DD1C, GND, R5, S1, SW1

Commit message: .
Parts:
- 1R1, 2R1, 3R1: value (none) -> 5k1
- 1RB: value (none) -> 47k&330k
- 1RG: value (none) -> 20k&120k
- 1RR: value (none) -> 470
- 2RB: value (none) -> 2k7&15k
- 2RG: value (none) -> 3k3
- 2RR: value (none) -> 3k8&150
- VT1, VT2, VT3: value KT3107 -> KT3107Ж
Connections:
- net 3V5 renamed 3V6
- net N$13 renamed G
- net N$14 renamed R
- net N$4 renamed B
Other:
- note added: "h=200..300"
- note added: "pin2 pwrled"
- note added: "pin3 pwrled"
- note added: "pin4 pwrled"
- note added: "pin6 pwron"
- note added: "pin8 pwron"
- moved on the sheet: 1R1, 1RB, 1RG, 1RR, 1VDB, 1VDG, 1VDR, 2R1, 2RB, 2RG, 2RR, 2VDB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
