File: pc2_usb3/pc2_usb.sch (EAGLE design)
At the start: 1 part, among them K1 692141030100

Commit message: .
Parts:
- added K2: 61400826021, Wurth_Elektronik_Electromechanic_Input-Output_Connectors_rev15c:61400826021
Changed lines of the file:
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@@
 <part name="FRAME1" library="frames" deviceset="DINA4_L" device=""/>
 <part name="K1" library="Wurth_Elektronik_Electromechanic_Input-Output_Connectors_rev15c" deviceset="692141030100" device=""/>
+<part name="K2" library="Wurth_Elektronik_Electromechanic_Input-Output_Connectors_rev15c" deviceset="61400826021" device=""/>
 </parts>
 <sheets>
@@
 <attribute name="VALUE" x="233.68" y="96.52" size="1.778" layer="96"/>
 </instance>
+<instance part="K2" gate="G$1" x="190.5" y="137.16"/>
 </instances>
 <busses>
