File: pc2_usb3/pc2_usb.brd (EAGLE design)
At the start: 1 part, among them K1 692141030100

Commit message: .
Parts:
- added K2: 61400826021, Wurth_Elektronik_Electromechanic_Input-Output_Connectors_rev15c:61400826021
- moved K1 5.20 mm to (15.9, 10.9)
Other:
- board outline added: 50 x 25 mm
Changed lines of the file:
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@@
 <setting verticaltext="up"/>
 </settings>
-<grid distance="50" unitdist="mil" unit="mil" style="lines" multiple="1" display="yes" altdistance="0.025" altunitdist="inch" altunit="inch"/>
+<grid distance="1" unitdist="mm" unit="mm" style="lines" multiple="1" display="yes" altdistance="0.025" altunitdist="inch" altunit="inch"/>
 <layers>
 <layer number="1" name="Top" color="4" fill="1" visible="yes" active="yes"/>
@@
 <board>
 <plain>
+<wire x1="2" y1="29" x2="52" y2="29" width="0.4064" layer="20"/>
+<wire x1="52" y1="29" x2="52" y2="4" width="0.4064" layer="20"/>
+<wire x1="52" y1="4" x2="2" y2="4" width="0.4064" layer="20"/>
+<wire x1="2" y1="4" x2="2" y2="29" width="0.4064" layer="20"/>
+<dimension x1="2" y1="33" x2="52" y2="33" x3="27" y3="42" textsize="1.778" layer="20" dtype="horizontal"/>
+<dimension x1="-2" y1="29" x2="-2" y2="4" x3="-15" y3="16.5" textsize="1.778" layer="20" dtype="vertical"/>
 </plain>
 <attributes>
@@
 </class>
 </classes>
-<designrules name="DesignRules">
-<description language="de">
-&lt;b&gt;EAGLE Design Rules&lt;/b&gt;
-</description>
-<description language="en">
-&lt;b&gt;EAGLE Design Rules&lt;/b&gt;
+<designrules name="pc2_usb">
+<description language="de">&lt;b&gt;EAGLE Design Rules&lt;/b&gt;
 &lt;p&gt;
-</description>
+Die Standard-Design-Rules sind so gewählt, dass sie für
+die meisten Anwendungen passen. Sollte ihre Platine
+besondere Anforderungen haben, treffen Sie die erforderlichen
+Einstellungen hier und speichern die Design Rules unter
+einem neuen Namen ab.</description>
+<description language="en">&lt;b&gt;EAGLE Design Rules&lt;/b&gt;
+&lt;p&gt;
+The default Design Rules have been set to cover
+a wide range of applications. Your particular design
+may have different requirements, so please make the
+necessary adjustments and save your customized
+design rules under a new name.</description>
 <param name="layerSetup" value="(1*16)"/>
 <param name="mtCopper" value="0.035mm 0.035mm 0.035mm 0.035mm 0.035mm 0.035mm 0.035mm 0.035mm 0.035mm 0.035mm 0.035mm 0.035mm 0.035mm 0.035mm 0.035mm 0.035mm"/>
 <param name="mtIsolate" value="1.5mm 0.15mm 0.2mm 0.15mm 0.2mm 0.15mm 0.2mm 0.15mm 0.2mm 0.15mm 0.2mm 0.15mm 0.2mm 0.15mm 0.2mm"/>
-<param name="mdWireWire" value="0.2mm"/>
-<param name="mdWirePad" value="0.2mm"/>
-<param name="mdWireVia" value="0.2mm"/>
+<param name="mdWireWire" value="8mil"/>
+<param name="mdWirePad" value="8mil"/>
+<param name="mdWireVia" value="8mil"/>
 <param name="mdPadPad" value="8mil"/>
 <param name="mdPadVia" value="8mil"/>
@@
 <param name="mdViaViaSameLayer" value="8mil"/>
 <param name="mnLayersViaInSmd" value="2"/>
-<param name="mdCopperDimension" value="10mil"/>
+<param name="mdCopperDimension" value="40mil"/>
 <param name="mdDrill" value="8mil"/>
 <param name="mdSmdStop" value="0mil"/>
-<param name="msWidth" value="8mil"/>
+<param name="msWidth" value="10mil"/>
 <param name="msDrill" value="24mil"/>
 <param name="msMicroVia" value="9.99mm"/>
 <param name="msBlindViaRatio" value="0.5"/>
-<param name="rvPadTop" value="0.2"/>
-<param name="rvPadInner" value="0.3"/>
-<param name="rvPadBottom" value="0.2"/>
+<param name="rvPadTop" value="0.25"/>
+<param name="rvPadInner" value="0.25"/>
+<param name="rvPadBottom" value="0.25"/>
 <param name="rvViaOuter" value="0.25"/>
 <param name="rvViaInner" value="0.25"/>
 <param name="rvMicroViaOuter" value="0.25"/>
 <param name="rvMicroViaInner" value="0.25"/>
-<param name="rlMinPadTop" value="0.5mm"/>
-<param name="rlMaxPadTop" value="1mm"/>
+<param name="rlMinPadTop" value="10mil"/>
+<param name="rlMaxPadTop" value="20mil"/>
 <param name="rlMinPadInner" value="10mil"/>
 <param name="rlMaxPadInner" value="20mil"/>
-<param name="rlMinPadBottom" value="0.5mm"/>
-<param name="rlMaxPadBottom" value="1mm"/>
+<param name="rlMinPadBottom" value="10mil"/>
+<param name="rlMaxPadBottom" value="20mil"/>
 <param name="rlMinViaOuter" value="8mil"/>
 <param name="rlMaxViaOuter" value="20mil"/>
@@
 </autorouter>
 <elements>
-<element name="K1" library="Wurth_Elektronik_Electromechanic_Input-Output_Connectors_rev15c" package="692141030100" value="692141030100" x="13.335" y="6.35" smashed="yes">
-<attribute name="VALUE" x="7.5475" y="16.0875" size="1.27" layer="27"/>
-<attribute name="NAME" x="11.9925" y="18.0875" size="1.27" layer="25"/>
+<element name="K1" library="Wurth_Elektronik_Electromechanic_Input-Output_Connectors_rev15c" package="692141030100" value="692141030100" x="15.875" y="10.89" smashed="yes">
+<attribute name="VALUE" x="10.0875" y="20.6275" size="1.27" layer="27"/>
+<attribute name="NAME" x="14.5325" y="22.6275" size="1.27" layer="25"/>
+</element>
+<element name="K2" library="Wurth_Elektronik_Electromechanic_Input-Output_Connectors_rev15c" package="61400826021" value="61400826021" x="40.005" y="17.5575" smashed="yes" rot="R180">
+<attribute name="NAME" x="38.753" y="25.051" size="1.27" layer="25"/>
+<attribute name="VALUE" x="34.943" y="19.1521" size="1.27" layer="27"/>
 </element>
 </elements>

Commit message: .
Parts:
- moved K2 1.00 mm to (41.0, 17.6)
Other:
- board size 50 x 25 mm -> 60 x 25 mm
Changed lines of the file:
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@@
 <board>
 <plain>
-<wire x1="2" y1="29" x2="52" y2="29" width="0.4064" layer="20"/>
-<wire x1="52" y1="29" x2="52" y2="4" width="0.4064" layer="20"/>
-<wire x1="52" y1="4" x2="2" y2="4" width="0.4064" layer="20"/>
-<wire x1="2" y1="4" x2="2" y2="29" width="0.4064" layer="20"/>
-<dimension x1="2" y1="33" x2="52" y2="33" x3="27" y3="42" textsize="1.778" layer="20" dtype="horizontal"/>
+<wire x1="-1" y1="29" x2="59" y2="29" width="0.4064" layer="20"/>
+<wire x1="59" y1="29" x2="59" y2="4" width="0.4064" layer="20"/>
+<wire x1="59" y1="4" x2="-1" y2="4" width="0.4064" layer="20"/>
+<wire x1="-1" y1="4" x2="-1" y2="29" width="0.4064" layer="20"/>
+<dimension x1="-1" y1="32" x2="59" y2="32" x3="29" y3="42" textsize="1.778" layer="20" dtype="horizontal"/>
 <dimension x1="-2" y1="29" x2="-2" y2="4" x3="-15" y3="16.5" textsize="1.778" layer="20" dtype="vertical"/>
+<dimension x1="49" y1="-8" x2="59" y2="-9" x3="54" y3="58" textsize="1.778" layer="20" dtype="horizontal"/>
 </plain>
 <attributes>
@@
 <attribute name="NAME" x="14.5325" y="22.6275" size="1.27" layer="25"/>
 </element>
-<element name="K2" library="Wurth_Elektronik_Electromechanic_Input-Output_Connectors_rev15c" package="61400826021" value="61400826021" x="40.005" y="17.5575" smashed="yes" rot="R180">
-<attribute name="NAME" x="38.753" y="25.051" size="1.27" layer="25"/>
-<attribute name="VALUE" x="34.943" y="19.1521" size="1.27" layer="27"/>
+<element name="K2" library="Wurth_Elektronik_Electromechanic_Input-Output_Connectors_rev15c" package="61400826021" value="61400826021" x="41.005" y="17.5575" smashed="yes" rot="R180">
+<attribute name="NAME" x="39.753" y="25.051" size="1.27" layer="25"/>
+<attribute name="VALUE" x="35.943" y="19.1521" size="1.27" layer="27"/>
 </element>
 </elements>
