File: pc2-key/pc2_key.brd (EAGLE design)
At the start: 98 x 35 mm, 56 parts, among them J2 0

Commit message: t2
Parts:
- added C3: 220n, resistor:C0805
- added R1: 470k, rcl:M0805
- 3RB: value 9k1&200k -> 470
- moved C8 0.64 mm to (8.26, 3.49)
- moved C7 0.63 mm to (14.3, 7.94)
- moved DD1 0.63 mm to (6.03, 14.3)
- moved SW1 0.63 mm to (-6.03, 9.53)
- moved !HDDLED 0.32 mm to (12.7, 15.6)
- moved GND 0.32 mm to (12.7, 20.6)
- moved PWRLED 0.32 mm to (12.7, 10.5)
Connections:
- removed net N$29: DD1.1, DD1.10, DD1.2
- new net N$13: C3.2, DD1.1, R1.2
- new net N$4: DD1.10, R1.1
- net PWRLED: now also DD1.2
- net VCC: now also C3.1
Routing:
- net N$29: track 9.74 -> 0.00 mm
- net N$4: track 0.00 -> 9.32 mm
- net !OUT_DSLED: track 75.0 -> 83.8 mm, vias 0 -> 2
- net VCC: track 84.6 -> 86.6 mm
- net PWRLED: track 7.19 -> 8.36 mm
- net N$21: track 9.35 -> 9.98 mm
- net GND: track 170.3 -> 171.0 mm
- net !OUT_PWLED: track 92.8 -> 93.3 mm
- net !DSKLED: track 8.31 -> 7.78 mm
Other:
- board text added: "HDD"
