File: pc2-key/pc2_key.sch (EAGLE design)
At the start: 52 parts, among them J2 0

Commit message: t2
Parts:
- added C3: 220n, resistor:C-EUC0805
- added R1: 470k, rcl:R-EU_M0805
- 3RB: value 9k1&200k -> 470
Connections:
- removed net N$29: DD1A.I0, DD1A.I1, DD1C.O
- new net N$13: C3.2, DD1A.I0, R1.2
- new net N$4: DD1C.O, R1.1
- net PWRLED: now also DD1A.I1
- net VCC: now also C3.1
Other:
- moved on the sheet: DD1A, DD1C, GND, R5, S1, SW1, ~{HDDLED}
